Commit message: add body meshes

File: install/rbt_simulation/share/rbt_simulation/robot/visual/otto-simulation.xacro (robot description, xacro)
@@ -8,5 +8,5 @@
             <origin rpy="0.0 0.0 0.0" xyz="0.0 0.0 0.0"/>
             <geometry>
-                <box size="0.13 0.15 0.13"/>
+              <mesh filename='package://rbt_simulation/meshes/Body.STL' scale="0.001 0.001 0.001"/>
             </geometry>
         </visual>

Commit message: leftleg

File: install/rbt_simulation/share/rbt_simulation/robot/visual/otto-simulation.xacro (robot description, xacro)
@@ -12,5 +12,5 @@
         </visual>
         <collision>
-            <origin rpy="0.0 0.0 0.0" xyz="0.0 0.0 0.3"/>
+            <origin rpy="0.0 0.0 0.0" xyz="0.0 0.0 0.0"/>
             <geometry>
                 <box size="0.13 0.15 0.13"/>
@@ -21,16 +21,34 @@
     <link name="hip_motorL">
         <visual>
-            <origin rpy="${PI/2} 0.0 0.0" xyz="0.0 0.0 0.0"/>
-            <geometry>
-                <cylinder radius="0.035" length="0.03"/>
+            <origin rpy="0.0 0.0 0.0" xyz="0.0 0.0 0.0"/>
+            <geometry>
+              <mesh filename='package://rbt_simulation/meshes/CyberGearmotor.STL' scale="0.001 0.001 0.001"/>
             </geometry>
         </visual>
+    </link>
+    <!-- Knee Motor Left -->
+    <link name="knee_motorL">
+      <visual>
+          <origin rpy="0.0 0.0 0.0" xyz="0.0 0.0 0.0"/>
+          <geometry>
+            <mesh filename='package://rbt_simulation/meshes/CyberGearmotor.STL' scale="0.001 0.001 0.001"/>
+          </geometry>
+      </visual>
+    </link>
+    <!-- Hip link Left -->
+    <link name="hip_linkL">
+      <visual>
+          <origin rpy="0.0 0.0 0.0" xyz="0.0 0.0 0.0"/>
+          <geometry>
+            <mesh filename='package://rbt_simulation/meshes/link1.STL' scale="0.001 0.001 0.001"/>
+          </geometry>
+      </visual>
     </link>
     <!-- Knee link Left -->
     <link name="knee_linkL">
       <visual>
-          <origin rpy="0.0 0.0 0.0" xyz="0.0 0.0 0.1"/>
-          <geometry>
-              <cylinder radius="0.01" length="0.2"/>
+          <origin rpy="${PI} ${-PI/2} 0.0" xyz="0.0 0.0 0.0"/>
+          <geometry>
+            <mesh filename='package://rbt_simulation/meshes/link2.STL' scale="0.001 0.001 0.001"/>
           </geometry>
       </visual>
@@ -39,7 +57,7 @@
     <link name="leg_linkL">
       <visual>
-          <origin rpy="0.0 0.0 0.0" xyz="0.0 0.0 0.1"/>
-          <geometry>
-              <cylinder radius="0.01" length="0.2"/>
+          <origin rpy="0.0 0.0 0.0" xyz="0.0 0.0 0.0"/>
+          <geometry>
+            <mesh filename='package://rbt_simulation/meshes/link4.STL' scale="0.001 0.001 0.001"/>
           </geometry>
       </visual>
@@ -48,7 +66,7 @@
     <link name="wheel_linkL">
       <visual>
-          <origin rpy="0.0 0.0 0.0" xyz="0.0 0.0 0.0"/>
-          <geometry>
-              <cylinder radius="0.1" length="0.025"/>
+          <origin rpy="${PI} 0.0 0.0" xyz="0.0 0.0 0.0"/>
+          <geometry>
+            <mesh filename='package://rbt_simulation/meshes/ODriveBotwheel.STL' scale="0.001 0.001 0.001"/>
           </geometry>
       </visual>
@@ -57,11 +75,23 @@
       <parent link="base_link"/>
       <child link="hip_motorL"/>
-        <origin rpy="0.0 ${-3*PI/4} 0.0" xyz="0.0 0.075 0.0"/>
+        <origin rpy="0.0 0.0 0.0" xyz="-0.03 0.06 0.0"/>
         <axis xyz="0.0 1.0 0.0"/>
     </joint>
+    <joint name="hip_motorL_to_knee_motorL" type="fixed">
+      <parent link="hip_motorL"/>
+      <child link="knee_motorL"/>
+      <origin rpy="0.0 0.0 0.0" xyz="0.0 0.05 0.0"/>
+      <axis xyz="0.0 1.0 0.0"/>
+    </joint>
+    <joint name="hip_motorL_to_hip_linkL" type="fixed">
+      <parent link="knee_motorL"/>
+      <child link="hip_linkL"/>
+      <origin rpy="0.0 0.0 0.0" xyz="0.0 0.035 0.0"/>
+      <axis xyz="0.0 1.0 0.0"/>
+    </joint>
     <joint name="hip_motorL_to_knee_linkL" type="continuous">
-      <parent link="hip_motorL"/>
+      <parent link="knee_motorL"/>
       <child link="knee_linkL"/>
-      <origin rpy="0.0 0.0 0.0" xyz="0.0 0.0 0.0"/>
+      <origin rpy="0.0 0.0 0.0" xyz="0.0 0.055 0.0"/>
       <axis xyz="0.0 1.0 0.0"/>
     </joint>
@@ -69,5 +99,5 @@
       <parent link="knee_linkL"/>
       <child link="leg_linkL"/>
-      <origin rpy="0.0 ${-PI/2} 0.0" xyz="0.0 0.0 0.2"/>
+      <origin rpy="0.0 0.0 0.0" xyz="-0.1414 -0.05 -0.1414"/>
       <axis xyz="0.0 1.0 0.0"/>
     </joint>
@@ -75,6 +105,6 @@
       <parent link="leg_linkL"/>
       <child link="wheel_linkL"/>
-      <origin rpy="${-PI/2} 0.0 0.0" xyz="0.0 0.0 0.2"/>
-      <axis xyz="0.0 0.0 0.1"/>
+      <origin rpy="0.0 0.0 0.0" xyz="0.1414 0.02 -0.1414"/>
+      <axis xyz="0.0 1.0 0.0"/>
     </joint>
     <!-- Right Side -->
@@ -82,16 +112,34 @@
     <link name="hip_motorR">
         <visual>
-            <origin rpy="${PI/2} 0.0 0.0" xyz="0.0 0.0 0.0"/>
-            <geometry>
-                <cylinder radius="0.035" length="0.03"/>
+            <origin rpy="${PI} 0.0 0.0" xyz="0.0 0.0 0.0"/>
+            <geometry>
+              <mesh filename='package://rbt_simulation/meshes/CyberGearmotor.STL' scale="0.001 0.001 0.001"/>
             </geometry>
         </visual>
+    </link>
+    <!-- Knee Motor Right -->
+    <link name="knee_motorR">
+      <visual>
+          <origin rpy="${PI} 0.0 0.0" xyz="0.0 0.0 0.0"/>
+          <geometry>
+            <mesh filename='package://rbt_simulation/meshes/CyberGearmotor.STL' scale="0.001 0.001 0.001"/>
+          </geometry>
+      </visual>
+    </link>
+    <!-- Hip link Right -->
+    <link name="hip_linkR">
+      <visual>
+          <origin rpy="0.0 0.0 0.0" xyz="0.0 0.0 0.0"/>
+          <geometry>
+            <mesh filename='package://rbt_simulation/meshes/link1R.STL' scale="0.001 0.001 0.001"/>
+          </geometry>
+      </visual>
     </link>
     <!-- Knee link Right -->
     <link name="knee_linkR">
       <visual>
-          <origin rpy="0.0 0.0 0.0" xyz="0.0 0.0 0.1"/>
-          <geometry>
-              <cylinder radius="0.01" length="0.2"/>
+          <origin rpy="0.0 0.0 0.0" xyz="0.0 0.0 0.0"/>
+          <geometry>
+            <mesh filename='package://rbt_simulation/meshes/link2R.STL' scale="0.001 0.001 0.001"/>
           </geometry>
       </visual>
@@ -100,7 +148,7 @@
     <link name="leg_linkR">
       <visual>
-          <origin rpy="0.0 0.0 0.0" xyz="0.0 0.0 0.1"/>
-          <geometry>
-              <cylinder radius="0.01" length="0.2"/>
+          <origin rpy="0.0 0.0 0.0" xyz="0.0 0.0 0.0"/>
+          <geometry>
+            <mesh filename='package://rbt_simulation/meshes/link4R.STL' scale="0.001 0.001 0.001"/>
           </geometry>
       </visual>
@@ -118,11 +166,23 @@
       <parent link="base_link"/>
       <child link="hip_motorR"/>
-        <origin rpy="0.0 ${-3*PI/4} 0.0" xyz="0.0 -0.075 0.0"/>
+        <origin rpy="0.0 0.0 0.0" xyz="-0.03 -0.06 0.0"/>
         <axis xyz="0.0 1.0 0.0"/>
     </joint>
+    <joint name="hip_motorR_to_knee_motorR" type="fixed">
+      <parent link="hip_motorR"/>
+      <child link="knee_motorR"/>
+        <origin rpy="0.0 0.0 0.0" xyz="0.0 -0.05 0.0"/>
+        <axis xyz="0.0 1.0 0.0"/>
+    </joint>
+    <joint name="hip_motorR_to_hip_linkR" type="fixed">
+      <parent link="knee_motorR"/>
+      <child link="hip_linkR"/>
+      <origin rpy="0.0 0.0 0.0" xyz="0.0 -0.035 0.0"/>
+      <axis xyz="0.0 1.0 0.0"/>
+    </joint>
     <joint name="hip_motorR_to_knee_linkR" type="continuous">
-      <parent link="hip_motorR"/>
+      <parent link="knee_motorR"/>
       <child link="knee_linkR"/>
-      <origin rpy="0.0 0.0 0.0" xyz="0.0 0.0 0.0"/>
+      <origin rpy="0.0 0.0 0.0" xyz="0.0 -0.05 0.0"/>
       <axis xyz="0.0 1.0 0.0"/>
     </joint>
@@ -130,5 +190,5 @@
       <parent link="knee_linkR"/>
       <child link="leg_linkR"/>
-      <origin rpy="0.0 ${-PI/2} 0.0" xyz="0.0 0.0 0.2"/>
+      <origin rpy="0.0 0.0 0.0" xyz="0.0 0.0 0.0"/>
       <axis xyz="0.0 1.0 0.0"/>
     </joint>

Commit message: urdf

File: install/rbt_simulation/share/rbt_simulation/robot/visual/otto-simulation.xacro (robot description, xacro)
@@ -72,5 +72,5 @@
       </visual>
     </link>
-    <joint name="base_to_hip_motorL" type="continuous">
+    <joint name="hip_jointL" type="continuous">
       <parent link="base_link"/>
       <child link="hip_motorL"/>
@@ -90,5 +90,5 @@
       <axis xyz="0.0 1.0 0.0"/>
     </joint>
-    <joint name="hip_motorL_to_knee_linkL" type="continuous">
+    <joint name="knee_jointL" type="continuous">
       <parent link="knee_motorL"/>
       <child link="knee_linkL"/>
@@ -96,11 +96,11 @@
       <axis xyz="0.0 1.0 0.0"/>
     </joint>
-    <joint name="knee_linkL_to_leg_linkL" type="continuous">
+    <joint name="virtualhip_jointL" type="continuous">
       <parent link="knee_linkL"/>
       <child link="leg_linkL"/>
-      <origin rpy="0.0 0.0 0.0" xyz="-0.1414 -0.05 -0.1414"/>
-      <axis xyz="0.0 1.0 0.0"/>
-    </joint>
-    <joint name="leg_linkL_wheel_linkL" type="continuous">
+      <origin rpy="0.0 0.0 0.0" xyz="-0.13718 -0.05 -0.14554"/>
+      <axis xyz="0.0 1.0 0.0"/>
+    </joint>
+    <joint name="wheel_jointL" type="continuous">
       <parent link="leg_linkL"/>
       <child link="wheel_linkL"/>
@@ -159,9 +159,9 @@
           <origin rpy="0.0 0.0 0.0" xyz="0.0 0.0 0.0"/>
           <geometry>
-              <cylinder radius="0.1" length="0.025"/>
-          </geometry>
-      </visual>
-    </link>
-    <joint name="base_to_hip_motorR" type="continuous">
+            <mesh filename='package://rbt_simulation/meshes/ODriveBotwheel.STL' scale="0.001 0.001 0.001"/>
+          </geometry>
+      </visual>
+    </link>
+    <joint name="hip_jointR" type="continuous">
       <parent link="base_link"/>
       <child link="hip_motorR"/>
@@ -181,5 +181,5 @@
       <axis xyz="0.0 1.0 0.0"/>
     </joint>
-    <joint name="hip_motorR_to_knee_linkR" type="continuous">
+    <joint name="knee_jointR" type="continuous">
       <parent link="knee_motorR"/>
       <child link="knee_linkR"/>
@@ -187,15 +187,15 @@
       <axis xyz="0.0 1.0 0.0"/>
     </joint>
-    <joint name="knee_linkR_to_leg_linkR" type="continuous">
+    <joint name="virtualhip_jointR" type="continuous">
       <parent link="knee_linkR"/>
       <child link="leg_linkR"/>
-      <origin rpy="0.0 0.0 0.0" xyz="0.0 0.0 0.0"/>
-      <axis xyz="0.0 1.0 0.0"/>
-    </joint>
-    <joint name="leg_linkR_wheel_linkR" type="continuous">
+      <origin rpy="0.0 0.0 0.0" xyz="-0.13718 0.05 -0.14554"/>
+      <axis xyz="0.0 1.0 0.0"/>
+    </joint>
+    <joint name="wheel_jointR" type="continuous">
       <parent link="leg_linkR"/>
       <child link="wheel_linkR"/>
-      <origin rpy="${-PI/2} 0.0 0.0" xyz="0.0 0.0 0.2"/>
-      <axis xyz="0.0 0.0 1.0"/>
+      <origin rpy="0.0 0.0 0.0" xyz="0.1414 -0.02 -0.1414"/>
+      <axis xyz="0.0 1.0 0.0"/>
     </joint>
 </robot>

Commit message: general launch

File: install/rbt_simulation/share/rbt_simulation/robot/visual/otto-simulation.xacro (robot description, xacro)
@@ -5,4 +5,9 @@
     <!-- Base Link -->
     <link name="base_link">
+        <inertial>
+          <origin xyz="-0.03 0.0 0.0" rpy="0 0 0"/>
+          <mass value="5.0"/>
+          <inertia ixx="0.553912" iyy="1.227224" izz="1.101448" ixy="-0.0" iyz="-0.0" ixz="0.005005"/>
+        </inertial>
         <visual>
             <origin rpy="0.0 0.0 0.0" xyz="0.0 0.0 0.0"/>
@@ -14,5 +19,5 @@
             <origin rpy="0.0 0.0 0.0" xyz="0.0 0.0 0.0"/>
             <geometry>
-                <box size="0.13 0.15 0.13"/>
+                <box size="0.20 0.19 0.15"/>
             </geometry>
         </collision>
@@ -48,5 +53,5 @@
     <link name="knee_linkL">
       <visual>
-          <origin rpy="${PI} ${-PI/2} 0.0" xyz="0.0 0.0 0.0"/>
+          <origin rpy="0.0 0.0 0.0" xyz="0.0 0.0 0.0"/>
           <geometry>
             <mesh filename='package://rbt_simulation/meshes/link2.STL' scale="0.001 0.001 0.001"/>
@@ -65,4 +70,9 @@
     <!-- wheel link Left -->
     <link name="wheel_linkL">
+      <inertial>
+        <origin xyz="0.0 0.02 0.0" rpy="0 0 0"/>
+        <mass value="1"/>
+        <inertia ixx="0.025678" iyy="0.046537" izz="0.025678" ixy="-0.0" iyz="0.0" ixz="0.0"/>
+      </inertial>
       <visual>
           <origin rpy="${PI} 0.0 0.0" xyz="0.0 0.0 0.0"/>
@@ -71,4 +81,10 @@
           </geometry>
       </visual>
+      <collision>
+        <origin rpy="${PI/2} 0.0 0.0" xyz="0.0 0.02 0.0"/>
+        <geometry>
+            <cylinder radius="0.086" length="0.04416"/>
+        </geometry>
+      </collision>
     </link>
     <joint name="hip_jointL" type="continuous">
@@ -99,5 +115,5 @@
       <parent link="knee_linkL"/>
       <child link="leg_linkL"/>
-      <origin rpy="0.0 0.0 0.0" xyz="-0.13718 -0.05 -0.14554"/>
+      <origin rpy="0.0 0.0 0.0" xyz="-0.1414 -0.05 -0.1414"/>
       <axis xyz="0.0 1.0 0.0"/>
     </joint>
@@ -156,4 +172,9 @@
     <!-- wheel link Right -->
     <link name="wheel_linkR">
+      <inertial>
+        <origin xyz="0.0 -0.02 0.0" rpy="0 0 0"/>
+        <mass value="1.0"/>
+        <inertia ixx="0.025678" iyy="0.046537" izz="0.025678" ixy="-0.0" iyz="0.0" ixz="0.0"/>
+      </inertial>
       <visual>
           <origin rpy="0.0 0.0 0.0" xyz="0.0 0.0 0.0"/>
@@ -162,4 +183,10 @@
           </geometry>
       </visual>
+      <collision>
+        <origin rpy="${PI/2} 0.0 0.0" xyz="0.0 -0.02 0.0"/>
+        <geometry>
+            <cylinder radius="0.086" length="0.04416"/>
+        </geometry>
+      </collision>
     </link>
     <joint name="hip_jointR" type="continuous">
@@ -190,5 +217,5 @@
       <parent link="knee_linkR"/>
       <child link="leg_linkR"/>
-      <origin rpy="0.0 0.0 0.0" xyz="-0.13718 0.05 -0.14554"/>
+      <origin rpy="0.0 0.0 0.0" xyz="-0.1414 0.05 -0.1414"/>
       <axis xyz="0.0 1.0 0.0"/>
     </joint>
