Commit message: cant spawn gazebo

File: install/otto_simulation/share/otto_simulation/urdf/otto-simulation.xacro (robot description, xacro)
@@ -1,6 +1,13 @@
 <?xml version="1.0"?>
-<robot xmlns:xacro="http://www.ros.org/wiki/xacro" name="example">
+<robot xmlns:xacro="http://www.ros.org/wiki/xacro" name="otto">
     <!-- Declare PI -->
     <xacro:property name="PI" value="3.14159265359"/>
+    <xacro:include filename="gazebo.xacro"/>
+    <link name="world"></link>
+    <joint name="base_joint" type="fixed">
+      <origin xyz="0 0 0.0" rpy="0 0 0"/>
+      <parent link="world"/>
+      <child link="base_link"/>
+    </joint>
     <!-- Base Link -->
     <link name="base_link">
@@ -25,13 +32,29 @@
     <!-- Hip Motor Left -->
     <link name="hip_motorL">
-        <visual>
-            <origin rpy="0.0 0.0 0.0" xyz="0.0 0.0 0.0"/>
-            <geometry>
-              <mesh filename='package://otto_simulation/meshes/CyberGearmotor.STL' scale="0.001 0.001 0.001"/>
-            </geometry>
-        </visual>
+      <inertial>
+        <origin xyz="0.00 0.0 0.0" rpy="0 0 0"/>
+        <mass value="2e-6"/>
+        <inertia ixx="1.1e-9" iyy="1.1e-9" izz="1.1e-9" ixy="0.0" iyz="0.0" ixz="0.0"/>
+      </inertial>
+      <visual>
+          <origin rpy="0.0 0.0 0.0" xyz="0.0 0.0 0.0"/>
+          <geometry>
+            <mesh filename='package://otto_simulation/meshes/CyberGearmotor.STL' scale="0.001 0.001 0.001"/>
+          </geometry>
+      </visual>
+      <collision>
+        <origin rpy="0.0 0.0 0.0" xyz="0.0 0.0 0.0"/>
+        <geometry>
+            <box size="1e-3 1e-3 1e-3"/>
+        </geometry>
+      </collision>
     </link>
     <!-- Knee Motor Left -->
     <link name="knee_motorL">
+      <inertial>
+        <origin xyz="0.00 0.0 0.0" rpy="0 0 0"/>
+        <mass value="2e-6"/>
+        <inertia ixx="1.1e-9" iyy="1.1e-9" izz="1.1e-9" ixy="0.0" iyz="0.0" ixz="0.0"/>
+      </inertial>
       <visual>
           <origin rpy="0.0 0.0 0.0" xyz="0.0 0.0 0.0"/>
@@ -40,7 +63,18 @@
           </geometry>
       </visual>
+      <collision>
+        <origin rpy="0.0 0.0 0.0" xyz="0.0 0.0 0.0"/>
+        <geometry>
+            <box size="1e-3 1e-3 1e-3"/>
+        </geometry>
+      </collision>
     </link>
     <!-- Hip link Left -->
     <link name="hip_linkL">
+      <inertial>
+        <origin xyz="0.00 0.0 0.0" rpy="0 0 0"/>
+        <mass value="2e-6"/>
+        <inertia ixx="1.1e-9" iyy="1.1e-9" izz="1.1e-9" ixy="0.0" iyz="0.0" ixz="0.0"/>
+      </inertial>
       <visual>
           <origin rpy="0.0 0.0 0.0" xyz="0.0 0.0 0.0"/>
@@ -49,7 +83,18 @@
           </geometry>
       </visual>
+      <collision>
+        <origin rpy="0.0 0.0 0.0" xyz="0.0 0.0 0.0"/>
+        <geometry>
+            <box size="1e-3 1e-3 1e-3"/>
+        </geometry>
+      </collision>
     </link>
     <!-- Knee link Left -->
     <link name="knee_linkL">
+      <inertial>
+        <origin xyz="0.00 0.0 0.0" rpy="0 0 0"/>
+        <mass value="2e-6"/>
+        <inertia ixx="1.1e-9" iyy="1.1e-9" izz="1.1e-9" ixy="0.0" iyz="0.0" ixz="0.0"/>
+      </inertial>
       <visual>
           <origin rpy="0.0 0.0 0.0" xyz="0.0 0.0 0.0"/>
@@ -58,7 +103,18 @@
           </geometry>
       </visual>
+      <collision>
+        <origin rpy="0.0 0.0 0.0" xyz="0.0 0.0 0.0"/>
+        <geometry>
+            <box size="1e-3 1e-3 1e-3"/>
+        </geometry>
+      </collision>
     </link>
     <!-- Leg link Left -->
     <link name="leg_linkL">
+      <inertial>
+        <origin xyz="0.00 0.0 0.0" rpy="0 0 0"/>
+        <mass value="2e-6"/>
+        <inertia ixx="1.1e-9" iyy="1.1e-9" izz="1.1e-9" ixy="0.0" iyz="0.0" ixz="0.0"/>
+      </inertial>
       <visual>
           <origin rpy="0.0 0.0 0.0" xyz="0.0 0.0 0.0"/>
@@ -67,4 +123,10 @@
           </geometry>
       </visual>
+      <collision>
+        <origin rpy="0.0 0.0 0.0" xyz="0.0 0.0 0.0"/>
+        <geometry>
+            <box size="1e-3 1e-3 1e-3"/>
+        </geometry>
+      </collision>
     </link>
     <!-- wheel link Left -->
@@ -127,13 +189,29 @@
     <!-- Hip Motor Right -->
     <link name="hip_motorR">
-        <visual>
-            <origin rpy="${PI} 0.0 0.0" xyz="0.0 0.0 0.0"/>
-            <geometry>
-              <mesh filename='package://otto_simulation/meshes/CyberGearmotor.STL' scale="0.001 0.001 0.001"/>
-            </geometry>
-        </visual>
+      <inertial>
+        <origin xyz="0.00 0.0 0.0" rpy="0 0 0"/>
+        <mass value="2e-6"/>
+        <inertia ixx="1.1e-9" iyy="1.1e-9" izz="1.1e-9" ixy="0.0" iyz="0.0" ixz="0.0"/>
+      </inertial>
+      <visual>
+          <origin rpy="${PI} 0.0 0.0" xyz="0.0 0.0 0.0"/>
+          <geometry>
+            <mesh filename='package://otto_simulation/meshes/CyberGearmotor.STL' scale="0.001 0.001 0.001"/>
+          </geometry>
+      </visual>
+      <collision>
+        <origin rpy="0.0 0.0 0.0" xyz="0.0 0.0 0.0"/>
+        <geometry>
+            <box size="1e-3 1e-3 1e-3"/>
+        </geometry>
+      </collision>
     </link>
     <!-- Knee Motor Right -->
     <link name="knee_motorR">
+      <inertial>
+        <origin xyz="0.00 0.0 0.0" rpy="0 0 0"/>
+        <mass value="2e-6"/>
+        <inertia ixx="1.1e-9" iyy="1.1e-9" izz="1.1e-9" ixy="0.0" iyz="0.0" ixz="0.0"/>
+      </inertial>
       <visual>
           <origin rpy="${PI} 0.0 0.0" xyz="0.0 0.0 0.0"/>
@@ -142,7 +220,18 @@
           </geometry>
       </visual>
+      <collision>
+        <origin rpy="0.0 0.0 0.0" xyz="0.0 0.0 0.0"/>
+        <geometry>
+            <box size="1e-3 1e-3 1e-3"/>
+        </geometry>
+      </collision>
     </link>
     <!-- Hip link Right -->
     <link name="hip_linkR">
+      <inertial>
+        <origin xyz="0.00 0.0 0.0" rpy="0 0 0"/>
+        <mass value="2e-6"/>
+        <inertia ixx="1.1e-9" iyy="1.1e-9" izz="1.1e-9" ixy="0.0" iyz="0.0" ixz="0.0"/>
+      </inertial>
       <visual>
           <origin rpy="0.0 0.0 0.0" xyz="0.0 0.0 0.0"/>
@@ -151,7 +240,18 @@
           </geometry>
       </visual>
+      <collision>
+        <origin rpy="0.0 0.0 0.0" xyz="0.0 0.0 0.0"/>
+        <geometry>
+            <box size="1e-3 1e-3 1e-3"/>
+        </geometry>
+      </collision>
     </link>
     <!-- Knee link Right -->
     <link name="knee_linkR">
+      <inertial>
+        <origin xyz="0.00 0.0 0.0" rpy="0 0 0"/>
+        <mass value="2e-6"/>
+        <inertia ixx="1.1e-9" iyy="1.1e-9" izz="1.1e-9" ixy="0.0" iyz="0.0" ixz="0.0"/>
+      </inertial>
       <visual>
           <origin rpy="0.0 0.0 0.0" xyz="0.0 0.0 0.0"/>
@@ -160,7 +260,18 @@
           </geometry>
       </visual>
+      <collision>
+        <origin rpy="0.0 0.0 0.0" xyz="0.0 0.0 0.0"/>
+        <geometry>
+            <box size="1e-3 1e-3 1e-3"/>
+        </geometry>
+      </collision>
     </link>
     <!-- Leg link Right -->
     <link name="leg_linkR">
+      <inertial>
+        <origin xyz="0.00 0.0 0.0" rpy="0 0 0"/>
+        <mass value="2e-6"/>
+        <inertia ixx="1.1e-9" iyy="1.1e-9" izz="1.1e-9" ixy="0.0" iyz="0.0" ixz="0.0"/>
+      </inertial>
       <visual>
           <origin rpy="0.0 0.0 0.0" xyz="0.0 0.0 0.0"/>
@@ -169,4 +280,10 @@
           </geometry>
       </visual>
+      <collision>
+        <origin rpy="0.0 0.0 0.0" xyz="0.0 0.0 0.0"/>
+        <geometry>
+            <box size="1e-3 1e-3 1e-3"/>
+        </geometry>
+      </collision>
     </link>
     <!-- wheel link Right -->
