Commit message: gazebo

File: install/otto_simulation/share/otto_simulation/urdf/gazebo.xacro (robot description, xacro)
@@ -6,9 +6,6 @@
         </hardware>
         <joint name="hip_jointL">
-            <command_interface name="position">
-                <param name="min">-3.14</param>
-                <param name="max">3.14</param>
-            </command_interface>
             <command_interface name="velocity"/>
+            <command_interface name="position"/>
             <state_interface name="position">
                 <param name="initial_value">0.0</param>
@@ -19,8 +16,5 @@
         <joint name="knee_jointL">
             <command_interface name="velocity"/>
-            <command_interface name="position">
-                <param name="min">-3.14</param>
-                <param name="max">3.14</param>
-            </command_interface>
+            <command_interface name="position"/>
             <state_interface name="position">
                 <param name="initial_value">0.0</param>
@@ -31,8 +25,5 @@
         <joint name="virtualhip_jointL">
             <command_interface name="velocity"/>
-            <command_interface name="position">
-                <param name="min">-3.14</param>
-                <param name="max">3.14</param>
-            </command_interface>
+            <command_interface name="position"/>
             <state_interface name="position">
                 <param name="initial_value">0.0</param>
@@ -43,8 +34,5 @@
         <joint name="wheel_jointL">
             <command_interface name="velocity"/>
-            <command_interface name="position">
-                <param name="min">-3.14</param>
-                <param name="max">3.14</param>
-            </command_interface>
+            <command_interface name="position"/>
             <state_interface name="position">
                 <param name="initial_value">0.0</param>
@@ -54,9 +42,6 @@
         </joint>
         <joint name="hip_jointR">
-            <command_interface name="position">
-                <param name="min">-3.14</param>
-                <param name="max">3.14</param>
-            </command_interface>
             <command_interface name="velocity"/>
+            <command_interface name="position"/>
             <state_interface name="position">
                 <param name="initial_value">0.0</param>
@@ -67,8 +52,5 @@
         <joint name="knee_jointR">
             <command_interface name="velocity"/>
-            <command_interface name="position">
-                <param name="min">-3.14</param>
-                <param name="max">3.14</param>
-            </command_interface>
+            <command_interface name="position"/>
             <state_interface name="position">
                 <param name="initial_value">0.0</param>
@@ -79,8 +61,5 @@
         <joint name="virtualhip_jointR">
             <command_interface name="velocity"/>
-            <command_interface name="position">
-                <param name="min">-3.14</param>
-                <param name="max">3.14</param>
-            </command_interface>
+            <command_interface name="position"/>
             <state_interface name="position">
                 <param name="initial_value">0.0</param>
@@ -91,8 +70,5 @@
         <joint name="wheel_jointR">
             <command_interface name="velocity"/>
-            <command_interface name="position">
-                <param name="min">-3.14</param>
-                <param name="max">3.14</param>
-            </command_interface>
+            <command_interface name="position"/>
             <state_interface name="position">
                 <param name="initial_value">0.0</param>
@@ -141,5 +117,4 @@
         <mu1>0.2</mu1>
         <mu2>0.2</mu2>
-        <material>Gazebo/Black</material>
     </gazebo>
     <gazebo reference="hip_motorR">
@@ -171,5 +146,4 @@
         <mu1>0.2</mu1>
         <mu2>0.2</mu2>
-        <material>Gazebo/Black</material>
     </gazebo>
 </robot>

File: install/otto_simulation/share/otto_simulation/urdf/otto-simulation.xacro (robot description, xacro)
@@ -6,5 +6,5 @@
     <link name="world"></link>
     <joint name="base_joint" type="fixed">
-      <origin xyz="0 0 0.0" rpy="0 0 0"/>
+      <origin xyz="0 0 0.4" rpy="0 0 0"/>
       <parent link="world"/>
       <child link="base_link"/>
@@ -20,5 +20,5 @@
             <origin rpy="0.0 0.0 0.0" xyz="0.0 0.0 0.0"/>
             <geometry>
-              <mesh filename='package://otto_simulation/meshes/Body.STL' scale="0.001 0.001 0.001"/>
+              <mesh filename='file:///$(find otto_simulation)/meshes/Body.STL' scale="0.001 0.001 0.001"/>
             </geometry>
         </visual>
@@ -40,13 +40,7 @@
           <origin rpy="0.0 0.0 0.0" xyz="0.0 0.0 0.0"/>
           <geometry>
-            <mesh filename='package://otto_simulation/meshes/CyberGearmotor.STL' scale="0.001 0.001 0.001"/>
-          </geometry>
-      </visual>
-      <collision>
-        <origin rpy="0.0 0.0 0.0" xyz="0.0 0.0 0.0"/>
-        <geometry>
-            <box size="1e-3 1e-3 1e-3"/>
-        </geometry>
-      </collision>
+            <mesh filename='file:///$(find otto_simulation)/meshes/CyberGearmotor.STL' scale="0.001 0.001 0.001"/>
+          </geometry>
+      </visual>
     </link>
     <!-- Knee Motor Left -->
@@ -60,13 +54,7 @@
           <origin rpy="0.0 0.0 0.0" xyz="0.0 0.0 0.0"/>
           <geometry>
-            <mesh filename='package://otto_simulation/meshes/CyberGearmotor.STL' scale="0.001 0.001 0.001"/>
-          </geometry>
-      </visual>
-      <collision>
-        <origin rpy="0.0 0.0 0.0" xyz="0.0 0.0 0.0"/>
-        <geometry>
-            <box size="1e-3 1e-3 1e-3"/>
-        </geometry>
-      </collision>
+            <mesh filename='file:///$(find otto_simulation)/meshes/CyberGearmotor.STL' scale="0.001 0.001 0.001"/>
+          </geometry>
+      </visual>
     </link>
     <!-- Hip link Left -->
@@ -80,13 +68,7 @@
           <origin rpy="0.0 0.0 0.0" xyz="0.0 0.0 0.0"/>
           <geometry>
-            <mesh filename='package://otto_simulation/meshes/link1.STL' scale="0.001 0.001 0.001"/>
-          </geometry>
-      </visual>
-      <collision>
-        <origin rpy="0.0 0.0 0.0" xyz="0.0 0.0 0.0"/>
-        <geometry>
-            <box size="1e-3 1e-3 1e-3"/>
-        </geometry>
-      </collision>
+            <mesh filename='file:///$(find otto_simulation)/meshes/link1.STL' scale="0.001 0.001 0.001"/>
+          </geometry>
+      </visual>
     </link>
     <!-- Knee link Left -->
@@ -100,13 +82,7 @@
           <origin rpy="0.0 0.0 0.0" xyz="0.0 0.0 0.0"/>
           <geometry>
-            <mesh filename='package://otto_simulation/meshes/link2.STL' scale="0.001 0.001 0.001"/>
-          </geometry>
-      </visual>
-      <collision>
-        <origin rpy="0.0 0.0 0.0" xyz="0.0 0.0 0.0"/>
-        <geometry>
-            <box size="1e-3 1e-3 1e-3"/>
-        </geometry>
-      </collision>
+            <mesh filename='file:///$(find otto_simulation)/meshes/link2.STL' scale="0.001 0.001 0.001"/>
+          </geometry>
+      </visual>
     </link>
     <!-- Leg link Left -->
@@ -120,13 +96,7 @@
           <origin rpy="0.0 0.0 0.0" xyz="0.0 0.0 0.0"/>
           <geometry>
-            <mesh filename='package://otto_simulation/meshes/link4.STL' scale="0.001 0.001 0.001"/>
-          </geometry>
-      </visual>
-      <collision>
-        <origin rpy="0.0 0.0 0.0" xyz="0.0 0.0 0.0"/>
-        <geometry>
-            <box size="1e-3 1e-3 1e-3"/>
-        </geometry>
-      </collision>
+            <mesh filename='file:///$(find otto_simulation)/meshes/link4.STL' scale="0.001 0.001 0.001"/>
+          </geometry>
+      </visual>
     </link>
     <!-- wheel link Left -->
@@ -140,5 +110,5 @@
           <origin rpy="${PI} 0.0 0.0" xyz="0.0 0.0 0.0"/>
           <geometry>
-            <mesh filename='package://otto_simulation/meshes/ODriveBotwheel.STL' scale="0.001 0.001 0.001"/>
+            <mesh filename='file:///$(find otto_simulation)/meshes/ODriveBotwheel.STL' scale="0.001 0.001 0.001"/>
           </geometry>
       </visual>
@@ -160,5 +130,4 @@
       <child link="knee_motorL"/>
       <origin rpy="0.0 0.0 0.0" xyz="0.0 0.05 0.0"/>
-      <axis xyz="0.0 1.0 0.0"/>
     </joint>
     <joint name="hip_motorL_to_hip_linkL" type="fixed">
@@ -166,5 +135,4 @@
       <child link="hip_linkL"/>
       <origin rpy="0.0 0.0 0.0" xyz="0.0 0.035 0.0"/>
-      <axis xyz="0.0 1.0 0.0"/>
     </joint>
     <joint name="knee_jointL" type="continuous">
@@ -197,13 +165,7 @@
           <origin rpy="${PI} 0.0 0.0" xyz="0.0 0.0 0.0"/>
           <geometry>
-            <mesh filename='package://otto_simulation/meshes/CyberGearmotor.STL' scale="0.001 0.001 0.001"/>
-          </geometry>
-      </visual>
-      <collision>
-        <origin rpy="0.0 0.0 0.0" xyz="0.0 0.0 0.0"/>
-        <geometry>
-            <box size="1e-3 1e-3 1e-3"/>
-        </geometry>
-      </collision>
+            <mesh filename='file:///$(find otto_simulation)/meshes/CyberGearmotor.STL' scale="0.001 0.001 0.001"/>
+          </geometry>
+      </visual>
     </link>
     <!-- Knee Motor Right -->
@@ -217,13 +179,7 @@
           <origin rpy="${PI} 0.0 0.0" xyz="0.0 0.0 0.0"/>
           <geometry>
-            <mesh filename='package://otto_simulation/meshes/CyberGearmotor.STL' scale="0.001 0.001 0.001"/>
-          </geometry>
-      </visual>
-      <collision>
-        <origin rpy="0.0 0.0 0.0" xyz="0.0 0.0 0.0"/>
-        <geometry>
-            <box size="1e-3 1e-3 1e-3"/>
-        </geometry>
-      </collision>
+            <mesh filename='file:///$(find otto_simulation)/meshes/CyberGearmotor.STL' scale="0.001 0.001 0.001"/>
+          </geometry>
+      </visual>
     </link>
     <!-- Hip link Right -->
@@ -237,13 +193,7 @@
           <origin rpy="0.0 0.0 0.0" xyz="0.0 0.0 0.0"/>
           <geometry>
-            <mesh filename='package://otto_simulation/meshes/link1R.STL' scale="0.001 0.001 0.001"/>
-          </geometry>
-      </visual>
-      <collision>
-        <origin rpy="0.0 0.0 0.0" xyz="0.0 0.0 0.0"/>
-        <geometry>
-            <box size="1e-3 1e-3 1e-3"/>
-        </geometry>
-      </collision>
+            <mesh filename='file:///$(find otto_simulation)/meshes/link1R.STL' scale="0.001 0.001 0.001"/>
+          </geometry>
+      </visual>
     </link>
     <!-- Knee link Right -->
@@ -257,13 +207,7 @@
           <origin rpy="0.0 0.0 0.0" xyz="0.0 0.0 0.0"/>
           <geometry>
-            <mesh filename='package://otto_simulation/meshes/link2R.STL' scale="0.001 0.001 0.001"/>
-          </geometry>
-      </visual>
-      <collision>
-        <origin rpy="0.0 0.0 0.0" xyz="0.0 0.0 0.0"/>
-        <geometry>
-            <box size="1e-3 1e-3 1e-3"/>
-        </geometry>
-      </collision>
+            <mesh filename='file:///$(find otto_simulation)/meshes/link2R.STL' scale="0.001 0.001 0.001"/>
+          </geometry>
+      </visual>
     </link>
     <!-- Leg link Right -->
@@ -277,13 +221,7 @@
           <origin rpy="0.0 0.0 0.0" xyz="0.0 0.0 0.0"/>
           <geometry>
-            <mesh filename='package://otto_simulation/meshes/link4R.STL' scale="0.001 0.001 0.001"/>
-          </geometry>
-      </visual>
-      <collision>
-        <origin rpy="0.0 0.0 0.0" xyz="0.0 0.0 0.0"/>
-        <geometry>
-            <box size="1e-3 1e-3 1e-3"/>
-        </geometry>
-      </collision>
+            <mesh filename='file:///$(find otto_simulation)/meshes/link4R.STL' scale="0.001 0.001 0.001"/>
+          </geometry>
+      </visual>
     </link>
     <!-- wheel link Right -->
@@ -297,5 +235,5 @@
           <origin rpy="0.0 0.0 0.0" xyz="0.0 0.0 0.0"/>
           <geometry>
-            <mesh filename='package://otto_simulation/meshes/ODriveBotwheel.STL' scale="0.001 0.001 0.001"/>
+            <mesh filename='file:///$(find otto_simulation)/meshes/ODriveBotwheel.STL' scale="0.001 0.001 0.001"/>
           </geometry>
       </visual>
@@ -317,5 +255,4 @@
       <child link="knee_motorR"/>
         <origin rpy="0.0 0.0 0.0" xyz="0.0 -0.05 0.0"/>
-        <axis xyz="0.0 1.0 0.0"/>
     </joint>
     <joint name="hip_motorR_to_hip_linkR" type="fixed">
@@ -323,5 +260,4 @@
       <child link="hip_linkR"/>
       <origin rpy="0.0 0.0 0.0" xyz="0.0 -0.035 0.0"/>
-      <axis xyz="0.0 1.0 0.0"/>
     </joint>
     <joint name="knee_jointR" type="continuous">
