Commit message: add innertia

File: install/otto_simulation/share/otto_simulation/urdf/gazebo.xacro (robot description, xacro)
@@ -1,5 +1,5 @@
 <?xml version="1.0"?>
 <robot xmlns:xacro="http://www.ros.org/wiki/xacro" name="otto">
-    <ros2_control name="GazeboSystem" type="system">
+    <!-- <ros2_control name="GazeboSystem" type="system">
         <hardware>
             <plugin>gazebo_ros2_control/GazeboSystem</plugin>
@@ -77,5 +77,5 @@
             <state_interface name="effort"/>
         </joint>
-    </ros2_control>
+    </ros2_control> -->
     <gazebo>
         <plugin filename="libgazebo_ros2_control.so" name="gazebo_ros2_control">

File: install/otto_simulation/share/otto_simulation/urdf/otto-simulation.xacro (robot description, xacro)
@@ -4,16 +4,20 @@
     <xacro:property name="PI" value="3.14159265359"/>
     <xacro:include filename="gazebo.xacro"/>
+    <xacro:include filename="inertial_macros.xacro"/>
+<!--
     <link name="world"></link>
     <joint name="base_joint" type="fixed">
-      <origin xyz="0 0 0.4" rpy="0 0 0"/>
+      <origin xyz="0 0 0.5" rpy="0 0 0"/>
       <parent link="world"/>
       <child link="base_link"/>
-    </joint>
+    </joint> -->
     <!-- Base Link -->
     <link name="base_link">
         <inertial>
-          <origin xyz="-0.03 0.0 0.0" rpy="0 0 0"/>
-          <mass value="5.0"/>
-          <inertia ixx="0.553912" iyy="1.227224" izz="1.101448" ixy="-0.0" iyz="-0.0" ixz="0.005005"/>
+          <origin xyz="0.0 0.0 0.0" rpy="0 0 0"/>
+          <mass value="5.21707"/>
+          <inertia ixx="25.36345483" ixy="0.0" ixz="-2.72079904"
+                   iyx="0.0" iyy="28.97825187" iyz="0.0"
+                   izx="-2.72079904" izy="0.0" izz="35.16013094" />
         </inertial>
         <visual>
@@ -33,7 +37,9 @@
     <link name="hip_motorL">
       <inertial>
-        <origin xyz="0.00 0.0 0.0" rpy="0 0 0"/>
-        <mass value="2e-6"/>
-        <inertia ixx="1.1e-9" iyy="1.1e-9" izz="1.1e-9" ixy="0.0" iyz="0.0" ixz="0.0"/>
+        <origin xyz="0.0 0.0 0.0" rpy="0 0 0"/>
+        <mass value="0.11255"/>
+        <inertia ixx="0.090104" ixy="0.000735" ixz="0.00035172"
+                 iyx="0.000735" iyy="0.074462" iyz="0.000140"
+                 izx="0.000351" izy="0.000140" izz="0.091432" />
       </inertial>
       <visual>
@@ -47,7 +53,9 @@
     <link name="knee_motorL">
       <inertial>
-        <origin xyz="0.00 0.0 0.0" rpy="0 0 0"/>
-        <mass value="2e-6"/>
-        <inertia ixx="1.1e-9" iyy="1.1e-9" izz="1.1e-9" ixy="0.0" iyz="0.0" ixz="0.0"/>
+        <origin xyz="0.0 0.0 0.0" rpy="0 0 0"/>
+        <mass value="0.11255"/>
+        <inertia ixx="0.090104" ixy="0.000735" ixz="0.00035172"
+                 iyx="0.000735" iyy="0.074462" iyz="0.000140"
+                 izx="0.000351" izy="0.000140" izz="0.091432" />
       </inertial>
       <visual>
@@ -61,7 +69,9 @@
     <link name="hip_linkL">
       <inertial>
-        <origin xyz="0.00 0.0 0.0" rpy="0 0 0"/>
-        <mass value="2e-6"/>
-        <inertia ixx="1.1e-9" iyy="1.1e-9" izz="1.1e-9" ixy="0.0" iyz="0.0" ixz="0.0"/>
+        <origin xyz="0.0 0.0 0.0" rpy="0 0 0"/>
+        <mass value="0.036"/>
+        <inertia ixx="0.038283" ixy="-0.00189" ixz="-0.020858"
+                 iyx="0.00189" iyy="0.066365" iyz="0.0021110"
+                 izx="0.0208580" izy="0.0021110" izz="0.030274" />
       </inertial>
       <visual>
@@ -75,7 +85,9 @@
     <link name="knee_linkL">
       <inertial>
-        <origin xyz="0.00 0.0 0.0" rpy="0 0 0"/>
-        <mass value="2e-6"/>
-        <inertia ixx="1.1e-9" iyy="1.1e-9" izz="1.1e-9" ixy="0.0" iyz="0.0" ixz="0.0"/>
+        <origin xyz="0.0 0.0 0.0" rpy="0 0 0"/>
+        <mass value="0.096"/>
+        <inertia ixx="0.808404" ixy="-0.054285" ixz="0.744011"
+                 iyx="-0.054285" iyy="1.51041728" iyz="-0.061449"
+                 izx="0.744011" izy="-0.061449" izz="0.743050" />
       </inertial>
       <visual>
@@ -89,7 +101,9 @@
     <link name="leg_linkL">
       <inertial>
-        <origin xyz="0.00 0.0 0.0" rpy="0 0 0"/>
-        <mass value="2e-6"/>
-        <inertia ixx="1.1e-9" iyy="1.1e-9" izz="1.1e-9" ixy="0.0" iyz="0.0" ixz="0.0"/>
+        <origin xyz="0.0 0.0 0.0" rpy="0 0 0"/>
+        <mass value="0.08537"/>
+        <inertia ixx="0.421600" ixy="0.022038" ixz="-0.474866"
+                 iyx="0.022038" iyy="0.982737" iyz="-0.017606"
+                 izx="-0.474866" izy="-0.017606" izz="0.566988" />
       </inertial>
       <visual>
@@ -103,7 +117,9 @@
     <link name="wheel_linkL">
       <inertial>
-        <origin xyz="0.0 0.02 0.0" rpy="0 0 0"/>
-        <mass value="1"/>
-        <inertia ixx="0.025678" iyy="0.046537" izz="0.025678" ixy="-0.0" iyz="0.0" ixz="0.0"/>
+        <origin xyz="0.0 0.0 0.0" rpy="0 0 0"/>
+        <mass value="0.51691"/>
+        <inertia ixx="1.717624" ixy="0.000049" ixz="-0.000006"
+                 iyx="0.000049" iyy="2.388020" iyz="0.000004"
+                 izx="-0.000006" izy="-0.000015" izz="1.717603" />
       </inertial>
       <visual>
@@ -120,5 +136,5 @@
       </collision>
     </link>
-    <joint name="hip_jointL" type="continuous">
+    <joint name="hip_jointL" type="fixed">
       <parent link="base_link"/>
       <child link="hip_motorL"/>
@@ -136,5 +152,5 @@
       <origin rpy="0.0 0.0 0.0" xyz="0.0 0.035 0.0"/>
     </joint>
-    <joint name="knee_jointL" type="continuous">
+    <joint name="knee_jointL" type="fixed">
       <parent link="knee_motorL"/>
       <child link="knee_linkL"/>
@@ -142,5 +158,5 @@
       <axis xyz="0.0 1.0 0.0"/>
     </joint>
-    <joint name="virtualhip_jointL" type="continuous">
+    <joint name="virtualhip_jointL" type="fixed">
       <parent link="knee_linkL"/>
       <child link="leg_linkL"/>
@@ -148,5 +164,5 @@
       <axis xyz="0.0 1.0 0.0"/>
     </joint>
-    <joint name="wheel_jointL" type="continuous">
+    <joint name="wheel_jointL" type="fixed">
       <parent link="leg_linkL"/>
       <child link="wheel_linkL"/>
@@ -158,7 +174,9 @@
     <link name="hip_motorR">
       <inertial>
-        <origin xyz="0.00 0.0 0.0" rpy="0 0 0"/>
-        <mass value="2e-6"/>
-        <inertia ixx="1.1e-9" iyy="1.1e-9" izz="1.1e-9" ixy="0.0" iyz="0.0" ixz="0.0"/>
+        <origin xyz="0.0 0.0 0.0" rpy="0 0 0"/>
+        <mass value="0.11255"/>
+        <inertia ixx="0.090104" ixy="0.000735" ixz="0.00035172"
+                 iyx="0.000735" iyy="0.074462" iyz="0.000140"
+                 izx="0.000351" izy="0.000140" izz="0.091432" />
       </inertial>
       <visual>
@@ -172,7 +190,9 @@
     <link name="knee_motorR">
       <inertial>
-        <origin xyz="0.00 0.0 0.0" rpy="0 0 0"/>
-        <mass value="2e-6"/>
-        <inertia ixx="1.1e-9" iyy="1.1e-9" izz="1.1e-9" ixy="0.0" iyz="0.0" ixz="0.0"/>
+        <origin xyz="0.0 0.0 0.0" rpy="0 0 0"/>
+        <mass value="0.096"/>
+        <inertia ixx="0.808404" ixy="0.054285" ixz="0.744011"
+                 iyx="0.054285" iyy="1.51041728" iyz="0.061449"
+                 izx="0.744011" izy="0.061449" izz="0.743050" />
       </inertial>
       <visual>
@@ -186,7 +206,9 @@
     <link name="hip_linkR">
       <inertial>
-        <origin xyz="0.00 0.0 0.0" rpy="0 0 0"/>
-        <mass value="2e-6"/>
-        <inertia ixx="1.1e-9" iyy="1.1e-9" izz="1.1e-9" ixy="0.0" iyz="0.0" ixz="0.0"/>
+        <origin xyz="0.0 0.0 0.0" rpy="0 0 0"/>
+        <mass value="0.036"/>
+        <inertia ixx="0.038283" ixy="0.00189" ixz="-0.020858"
+                 iyx="0.00189" iyy="0.066365" iyz="-0.0021110"
+                 izx="-0.0208580" izy="-0.0021110" izz="0.030274" />
       </inertial>
       <visual>
@@ -200,7 +222,9 @@
     <link name="knee_linkR">
       <inertial>
-        <origin xyz="0.00 0.0 0.0" rpy="0 0 0"/>
-        <mass value="2e-6"/>
-        <inertia ixx="1.1e-9" iyy="1.1e-9" izz="1.1e-9" ixy="0.0" iyz="0.0" ixz="0.0"/>
+        <origin xyz="0.0 0.0 0.0" rpy="0 0 0"/>
+        <mass value="0.096"/>
+        <inertia ixx="0.808404" ixy="0.054285" ixz="0.744011"
+                 iyx="0.054285" iyy="1.51041728" iyz="0.061449"
+                 izx="0.744011" izy="-0.061449" izz="0.743050" />
       </inertial>
       <visual>
@@ -214,7 +238,9 @@
     <link name="leg_linkR">
       <inertial>
-        <origin xyz="0.00 0.0 0.0" rpy="0 0 0"/>
-        <mass value="2e-6"/>
-        <inertia ixx="1.1e-9" iyy="1.1e-9" izz="1.1e-9" ixy="0.0" iyz="0.0" ixz="0.0"/>
+        <origin xyz="0.0 0.0 0.0" rpy="0 0 0"/>
+        <mass value="0.08537"/>
+        <inertia ixx="0.421600" ixy="-0.022038" ixz="-0.474866"
+                 iyx="-0.022038" iyy="0.982737" iyz="0.017606"
+                 izx="-0.474866" izy="0.017606" izz="0.566988" />
       </inertial>
       <visual>
@@ -228,7 +254,9 @@
     <link name="wheel_linkR">
       <inertial>
-        <origin xyz="0.0 -0.02 0.0" rpy="0 0 0"/>
-        <mass value="1.0"/>
-        <inertia ixx="0.025678" iyy="0.046537" izz="0.025678" ixy="-0.0" iyz="0.0" ixz="0.0"/>
+        <origin xyz="0.0 0.0 0.0" rpy="0 0 0"/>
+        <mass value="0.51691"/>
+        <inertia ixx="1.717624" ixy="0.000049" ixz="-0.000006"
+                 iyx="0.000049" iyy="2.388020" iyz="0.000004"
+                 izx="-0.000006" izy="-0.000015" izz="1.717603" />
       </inertial>
       <visual>
@@ -245,5 +273,5 @@
       </collision>
     </link>
-    <joint name="hip_jointR" type="continuous">
+    <joint name="hip_jointR" type="fixed">
       <parent link="base_link"/>
       <child link="hip_motorR"/>
@@ -261,5 +289,5 @@
       <origin rpy="0.0 0.0 0.0" xyz="0.0 -0.035 0.0"/>
     </joint>
-    <joint name="knee_jointR" type="continuous">
+    <joint name="knee_jointR" type="fixed">
       <parent link="knee_motorR"/>
       <child link="knee_linkR"/>
@@ -267,5 +295,5 @@
       <axis xyz="0.0 1.0 0.0"/>
     </joint>
-    <joint name="virtualhip_jointR" type="continuous">
+    <joint name="virtualhip_jointR" type="fixed">
       <parent link="knee_linkR"/>
       <child link="leg_linkR"/>
@@ -273,5 +301,5 @@
       <axis xyz="0.0 1.0 0.0"/>
     </joint>
-    <joint name="wheel_jointR" type="continuous">
+    <joint name="wheel_jointR" type="fixed">
       <parent link="leg_linkR"/>
       <child link="wheel_linkR"/>

File: src/otto_simulation/urdf/otto-simulation.xacro (robot description, xacro)
@@ -4,7 +4,8 @@
     <xacro:property name="PI" value="3.14159265359"/>
     <xacro:include filename="gazebo.xacro"/>
+    <xacro:include filename="inertial_macros.xacro"/>
     <link name="world"></link>
     <joint name="base_joint" type="fixed">
-      <origin xyz="0 0 0.4" rpy="0 0 0"/>
+      <origin xyz="0 0 0.5" rpy="0 0 0"/>
       <parent link="world"/>
       <child link="base_link"/>
@@ -13,7 +14,9 @@
     <link name="base_link">
         <inertial>
-          <origin xyz="-0.03 0.0 0.0" rpy="0 0 0"/>
-          <mass value="5.0"/>
-          <inertia ixx="0.553912" iyy="1.227224" izz="1.101448" ixy="-0.0" iyz="-0.0" ixz="0.005005"/>
+          <origin xyz="0.0 0.0 0.0" rpy="0 0 0"/>
+          <mass value="5.21707"/>
+          <inertia ixx="25.36345483" ixy="0.0" ixz="-2.72079904"
+                   iyx="0.0" iyy="28.97825187" iyz="0.0"
+                   izx="-2.72079904" izy="0.0" izz="35.16013094" />
         </inertial>
         <visual>
@@ -33,7 +36,9 @@
     <link name="hip_motorL">
       <inertial>
-        <origin xyz="0.00 0.0 0.0" rpy="0 0 0"/>
-        <mass value="2e-6"/>
-        <inertia ixx="1.1e-9" iyy="1.1e-9" izz="1.1e-9" ixy="0.0" iyz="0.0" ixz="0.0"/>
+        <origin xyz="0.0 0.0 0.0" rpy="0 0 0"/>
+        <mass value="0.11255"/>
+        <inertia ixx="0.090104" ixy="0.000735" ixz="0.00035172"
+                 iyx="0.000735" iyy="0.074462" iyz="0.000140"
+                 izx="0.000351" izy="0.000140" izz="0.091432" />
       </inertial>
       <visual>
@@ -47,7 +52,9 @@
     <link name="knee_motorL">
       <inertial>
-        <origin xyz="0.00 0.0 0.0" rpy="0 0 0"/>
-        <mass value="2e-6"/>
-        <inertia ixx="1.1e-9" iyy="1.1e-9" izz="1.1e-9" ixy="0.0" iyz="0.0" ixz="0.0"/>
+        <origin xyz="0.0 0.0 0.0" rpy="0 0 0"/>
+        <mass value="0.11255"/>
+        <inertia ixx="0.090104" ixy="0.000735" ixz="0.00035172"
+                 iyx="0.000735" iyy="0.074462" iyz="0.000140"
+                 izx="0.000351" izy="0.000140" izz="0.091432" />
       </inertial>
       <visual>
@@ -61,7 +68,9 @@
     <link name="hip_linkL">
       <inertial>
-        <origin xyz="0.00 0.0 0.0" rpy="0 0 0"/>
-        <mass value="2e-6"/>
-        <inertia ixx="1.1e-9" iyy="1.1e-9" izz="1.1e-9" ixy="0.0" iyz="0.0" ixz="0.0"/>
+        <origin xyz="0.0 0.0 0.0" rpy="0 0 0"/>
+        <mass value="0.036"/>
+        <inertia ixx="0.038283" ixy="-0.00189" ixz="-0.020858"
+                 iyx="0.00189" iyy="0.066365" iyz="0.0021110"
+                 izx="0.0208580" izy="0.0021110" izz="0.030274" />
       </inertial>
       <visual>
@@ -75,7 +84,9 @@
     <link name="knee_linkL">
       <inertial>
-        <origin xyz="0.00 0.0 0.0" rpy="0 0 0"/>
-        <mass value="2e-6"/>
-        <inertia ixx="1.1e-9" iyy="1.1e-9" izz="1.1e-9" ixy="0.0" iyz="0.0" ixz="0.0"/>
+        <origin xyz="0.0 0.0 0.0" rpy="0 0 0"/>
+        <mass value="0.096"/>
+        <inertia ixx="0.808404" ixy="-0.054285" ixz="0.744011"
+                 iyx="-0.054285" iyy="1.51041728" iyz="-0.061449"
+                 izx="0.744011" izy="-0.061449" izz="0.743050" />
       </inertial>
       <visual>
@@ -89,7 +100,9 @@
     <link name="leg_linkL">
       <inertial>
-        <origin xyz="0.00 0.0 0.0" rpy="0 0 0"/>
-        <mass value="2e-6"/>
-        <inertia ixx="1.1e-9" iyy="1.1e-9" izz="1.1e-9" ixy="0.0" iyz="0.0" ixz="0.0"/>
+        <origin xyz="0.0 0.0 0.0" rpy="0 0 0"/>
+        <mass value="0.08537"/>
+        <inertia ixx="0.421600" ixy="0.022038" ixz="-0.474866"
+                 iyx="0.022038" iyy="0.982737" iyz="-0.017606"
+                 izx="-0.474866" izy="-0.017606" izz="0.566988" />
       </inertial>
       <visual>
@@ -103,7 +116,9 @@
     <link name="wheel_linkL">
       <inertial>
-        <origin xyz="0.0 0.02 0.0" rpy="0 0 0"/>
-        <mass value="1"/>
-        <inertia ixx="0.025678" iyy="0.046537" izz="0.025678" ixy="-0.0" iyz="0.0" ixz="0.0"/>
+        <origin xyz="0.0 0.0 0.0" rpy="0 0 0"/>
+        <mass value="0.51691"/>
+        <inertia ixx="1.717624" ixy="0.000049" ixz="-0.000006"
+                 iyx="0.000049" iyy="2.388020" iyz="0.000004"
+                 izx="-0.000006" izy="-0.000015" izz="1.717603" />
       </inertial>
       <visual>
@@ -158,7 +173,9 @@
     <link name="hip_motorR">
       <inertial>
-        <origin xyz="0.00 0.0 0.0" rpy="0 0 0"/>
-        <mass value="2e-6"/>
-        <inertia ixx="1.1e-9" iyy="1.1e-9" izz="1.1e-9" ixy="0.0" iyz="0.0" ixz="0.0"/>
+        <origin xyz="0.0 0.0 0.0" rpy="0 0 0"/>
+        <mass value="0.11255"/>
+        <inertia ixx="0.090104" ixy="0.000735" ixz="0.00035172"
+                 iyx="0.000735" iyy="0.074462" iyz="0.000140"
+                 izx="0.000351" izy="0.000140" izz="0.091432" />
       </inertial>
       <visual>
@@ -172,7 +189,9 @@
     <link name="knee_motorR">
       <inertial>
-        <origin xyz="0.00 0.0 0.0" rpy="0 0 0"/>
-        <mass value="2e-6"/>
-        <inertia ixx="1.1e-9" iyy="1.1e-9" izz="1.1e-9" ixy="0.0" iyz="0.0" ixz="0.0"/>
+        <origin xyz="0.0 0.0 0.0" rpy="0 0 0"/>
+        <mass value="0.096"/>
+        <inertia ixx="0.808404" ixy="0.054285" ixz="0.744011"
+                 iyx="0.054285" iyy="1.51041728" iyz="0.061449"
+                 izx="0.744011" izy="0.061449" izz="0.743050" />
       </inertial>
       <visual>
@@ -186,7 +205,9 @@
     <link name="hip_linkR">
       <inertial>
-        <origin xyz="0.00 0.0 0.0" rpy="0 0 0"/>
-        <mass value="2e-6"/>
-        <inertia ixx="1.1e-9" iyy="1.1e-9" izz="1.1e-9" ixy="0.0" iyz="0.0" ixz="0.0"/>
+        <origin xyz="0.0 0.0 0.0" rpy="0 0 0"/>
+        <mass value="0.036"/>
+        <inertia ixx="0.038283" ixy="0.00189" ixz="-0.020858"
+                 iyx="0.00189" iyy="0.066365" iyz="-0.0021110"
+                 izx="-0.0208580" izy="-0.0021110" izz="0.030274" />
       </inertial>
       <visual>
@@ -200,7 +221,9 @@
     <link name="knee_linkR">
       <inertial>
-        <origin xyz="0.00 0.0 0.0" rpy="0 0 0"/>
-        <mass value="2e-6"/>
-        <inertia ixx="1.1e-9" iyy="1.1e-9" izz="1.1e-9" ixy="0.0" iyz="0.0" ixz="0.0"/>
+        <origin xyz="0.0 0.0 0.0" rpy="0 0 0"/>
+        <mass value="0.096"/>
+        <inertia ixx="0.808404" ixy="0.054285" ixz="0.744011"
+                 iyx="0.054285" iyy="1.51041728" iyz="0.061449"
+                 izx="0.744011" izy="-0.061449" izz="0.743050" />
       </inertial>
       <visual>
@@ -214,7 +237,9 @@
     <link name="leg_linkR">
       <inertial>
-        <origin xyz="0.00 0.0 0.0" rpy="0 0 0"/>
-        <mass value="2e-6"/>
-        <inertia ixx="1.1e-9" iyy="1.1e-9" izz="1.1e-9" ixy="0.0" iyz="0.0" ixz="0.0"/>
+        <origin xyz="0.0 0.0 0.0" rpy="0 0 0"/>
+        <mass value="0.08537"/>
+        <inertia ixx="0.421600" ixy="-0.022038" ixz="-0.474866"
+                 iyx="-0.022038" iyy="0.982737" iyz="0.017606"
+                 izx="-0.474866" izy="0.017606" izz="0.566988" />
       </inertial>
       <visual>
@@ -228,7 +253,9 @@
     <link name="wheel_linkR">
       <inertial>
-        <origin xyz="0.0 -0.02 0.0" rpy="0 0 0"/>
-        <mass value="1.0"/>
-        <inertia ixx="0.025678" iyy="0.046537" izz="0.025678" ixy="-0.0" iyz="0.0" ixz="0.0"/>
+        <origin xyz="0.0 0.0 0.0" rpy="0 0 0"/>
+        <mass value="0.51691"/>
+        <inertia ixx="1.717624" ixy="0.000049" ixz="-0.000006"
+                 iyx="0.000049" iyy="2.388020" iyz="0.000004"
+                 izx="-0.000006" izy="-0.000015" izz="1.717603" />
       </inertial>
       <visual>
