Commit message: gitignore

File: install/otto_simulation/share/otto_simulation/urdf/gazebo.xacro (robot description, xacro)
@@ -1,10 +1,9 @@
 <?xml version="1.0"?>
 <robot xmlns:xacro="http://www.ros.org/wiki/xacro" name="otto">
-    <!-- <ros2_control name="GazeboSystem" type="system">
+    <ros2_control name="GazeboSystem" type="system">
         <hardware>
             <plugin>gazebo_ros2_control/GazeboSystem</plugin>
         </hardware>
         <joint name="hip_jointL">
-            <command_interface name="velocity"/>
             <command_interface name="position"/>
             <state_interface name="position">
@@ -15,5 +14,4 @@
         </joint>
         <joint name="knee_jointL">
-            <command_interface name="velocity"/>
             <command_interface name="position"/>
             <state_interface name="position">
@@ -24,5 +22,4 @@
         </joint>
         <joint name="virtualhip_jointL">
-            <command_interface name="velocity"/>
             <command_interface name="position"/>
             <state_interface name="position">
@@ -33,5 +30,4 @@
         </joint>
         <joint name="wheel_jointL">
-            <command_interface name="velocity"/>
             <command_interface name="position"/>
             <state_interface name="position">
@@ -42,5 +38,4 @@
         </joint>
         <joint name="hip_jointR">
-            <command_interface name="velocity"/>
             <command_interface name="position"/>
             <state_interface name="position">
@@ -51,5 +46,4 @@
         </joint>
         <joint name="knee_jointR">
-            <command_interface name="velocity"/>
             <command_interface name="position"/>
             <state_interface name="position">
@@ -60,5 +54,4 @@
         </joint>
         <joint name="virtualhip_jointR">
-            <command_interface name="velocity"/>
             <command_interface name="position"/>
             <state_interface name="position">
@@ -69,5 +62,4 @@
         </joint>
         <joint name="wheel_jointR">
-            <command_interface name="velocity"/>
             <command_interface name="position"/>
             <state_interface name="position">
@@ -77,5 +69,5 @@
             <state_interface name="effort"/>
         </joint>
-    </ros2_control> -->
+    </ros2_control>
     <gazebo>
         <plugin filename="libgazebo_ros2_control.so" name="gazebo_ros2_control">

File: install/otto_simulation/share/otto_simulation/urdf/otto-simulation.xacro (robot description, xacro)
@@ -4,9 +4,7 @@
     <xacro:property name="PI" value="3.14159265359"/>
     <xacro:include filename="gazebo.xacro"/>
-    <xacro:include filename="inertial_macros.xacro"/>
-<!--
-    <link name="world"></link>
+    <!-- <link name="world"></link>
     <joint name="base_joint" type="fixed">
-      <origin xyz="0 0 0.5" rpy="0 0 0"/>
+      <origin xyz="0 0 0.0" rpy="0 0 0"/>
       <parent link="world"/>
       <child link="base_link"/>
@@ -136,9 +134,10 @@
       </collision>
     </link>
-    <joint name="hip_jointL" type="fixed">
+    <joint name="hip_jointL" type="continuous">
       <parent link="base_link"/>
       <child link="hip_motorL"/>
         <origin rpy="0.0 0.0 0.0" xyz="-0.03 0.06 0.0"/>
         <axis xyz="0.0 1.0 0.0"/>
+      <dynamics damping="0.1" friction="0.05"/>
     </joint>
     <joint name="hip_motorL_to_knee_motorL" type="fixed">
@@ -152,21 +151,24 @@
       <origin rpy="0.0 0.0 0.0" xyz="0.0 0.035 0.0"/>
     </joint>
-    <joint name="knee_jointL" type="fixed">
+    <joint name="knee_jointL" type="continuous">
       <parent link="knee_motorL"/>
       <child link="knee_linkL"/>
       <origin rpy="0.0 0.0 0.0" xyz="0.0 0.055 0.0"/>
       <axis xyz="0.0 1.0 0.0"/>
-    </joint>
-    <joint name="virtualhip_jointL" type="fixed">
+      <dynamics damping="0.1" friction="0.05"/>
+    </joint>
+    <joint name="virtualhip_jointL" type="continuous">
       <parent link="knee_linkL"/>
       <child link="leg_linkL"/>
       <origin rpy="0.0 0.0 0.0" xyz="-0.1414 -0.05 -0.1414"/>
       <axis xyz="0.0 1.0 0.0"/>
-    </joint>
-    <joint name="wheel_jointL" type="fixed">
+      <dynamics damping="0.1" friction="0.05"/>
+    </joint>
+    <joint name="wheel_jointL" type="continuous">
       <parent link="leg_linkL"/>
       <child link="wheel_linkL"/>
       <origin rpy="0.0 0.0 0.0" xyz="0.1414 0.02 -0.1414"/>
       <axis xyz="0.0 1.0 0.0"/>
+      <dynamics damping="0.1" friction="0.05"/>
     </joint>
     <!-- Right Side -->
@@ -273,9 +275,10 @@
       </collision>
     </link>
-    <joint name="hip_jointR" type="fixed">
+    <joint name="hip_jointR" type="continuous">
       <parent link="base_link"/>
       <child link="hip_motorR"/>
         <origin rpy="0.0 0.0 0.0" xyz="-0.03 -0.06 0.0"/>
         <axis xyz="0.0 1.0 0.0"/>
+        <dynamics damping="0.1" friction="0.05"/>
     </joint>
     <joint name="hip_motorR_to_knee_motorR" type="fixed">
@@ -289,21 +292,24 @@
       <origin rpy="0.0 0.0 0.0" xyz="0.0 -0.035 0.0"/>
     </joint>
-    <joint name="knee_jointR" type="fixed">
+    <joint name="knee_jointR" type="continuous">
       <parent link="knee_motorR"/>
       <child link="knee_linkR"/>
       <origin rpy="0.0 0.0 0.0" xyz="0.0 -0.05 0.0"/>
       <axis xyz="0.0 1.0 0.0"/>
-    </joint>
-    <joint name="virtualhip_jointR" type="fixed">
+      <dynamics damping="0.1" friction="0.05"/>
+    </joint>
+    <joint name="virtualhip_jointR" type="continuous">
       <parent link="knee_linkR"/>
       <child link="leg_linkR"/>
       <origin rpy="0.0 0.0 0.0" xyz="-0.1414 0.05 -0.1414"/>
       <axis xyz="0.0 1.0 0.0"/>
-    </joint>
-    <joint name="wheel_jointR" type="fixed">
+      <dynamics damping="0.1" friction="0.05"/>
+    </joint>
+    <joint name="wheel_jointR" type="continuous">
       <parent link="leg_linkR"/>
       <child link="wheel_linkR"/>
       <origin rpy="0.0 0.0 0.0" xyz="0.1414 -0.02 -0.1414"/>
       <axis xyz="0.0 1.0 0.0"/>
+      <dynamics damping="0.1" friction="0.05"/>
     </joint>
 </robot>

File: src/otto_simulation/urdf/otto-simulation.urdf (robot description, URDF)
Before this commit: robot otto, 14 links, 13 joints
Links:
- removed link world
- link base_link: mass 5.21707 -> None
Joints:
- removed joint base_joint
