Commit message: pid

File: otto_simulation/urdf/otto-simulationtest.xacro (robot description, xacro)
@@ -3,5 +3,5 @@
     <!-- Declare PI -->
     <xacro:property name="PI" value="3.14159265359"/>
-    <xacro:include filename="gazebo.xacro"/>
+    <xacro:include filename="gazebotest.xacro"/>
     <!-- <link name="world"></link>
     <joint name="base_joint" type="fixed">
@@ -13,6 +13,6 @@
     <link name="base_link">
         <inertial>
-          <origin xyz="0.0 0.0 0.0" rpy="0 0 0"/>
-          <mass value="5.217065"/>
+          <origin xyz="-0.025374 0.0 0.0" rpy="0 0 0"/>
+          <mass value="5.21707"/>
           <inertia ixx="25.36345483e-3" ixy="0.0" ixz="-2.72079904e-3"
                    iyx="0.0" iyy="28.97825187e-3" iyz="0.0"
@@ -149,5 +149,5 @@
       </collision>
     </link>
-    <joint name="hip_jointL" type="revolute">
+    <joint name="hip_jointL" type="fixed">
       <parent link="base_link"/>
       <child link="hip_motorL"/>
@@ -155,5 +155,5 @@
         <axis xyz="0.0 1.0 0.0"/>
       <dynamics damping="0.2" friction="0.05"/>
-      <limit effort="15.0" lower="${-PI}" upper="${PI}" velocity="30"/>
+      <limit effort="50.0" lower="${-PI}" upper="${PI}" velocity="30"/>
     </joint>
     <joint name="hip_motorL_to_knee_motorL" type="fixed">
@@ -167,5 +167,5 @@
       <origin rpy="0.0 0.0 0.0" xyz="0.0 0.035 0.0"/>
     </joint>
-    <joint name="knee_jointL" type="revolute">
+    <joint name="knee_jointL" type="fixed">
       <parent link="knee_motorL"/>
       <child link="knee_linkL"/>
@@ -173,7 +173,7 @@
       <axis xyz="0.0 1.0 0.0"/>
       <dynamics damping="0.1" friction="0.02"/>
-      <limit effort="15.0" lower="${-PI}" upper="${PI}" velocity="30"/>
-    </joint>
-    <joint name="virtualhip_jointL" type="revolute">
+      <limit effort="50.0" lower="${-PI}" upper="${PI}" velocity="30"/>
+    </joint>
+    <joint name="virtualhip_jointL" type="fixed">
       <parent link="knee_linkL"/>
       <child link="leg_linkL"/>
@@ -181,5 +181,5 @@
       <axis xyz="0.0 1.0 0.0"/>
       <dynamics damping="0.1" friction="0.05"/>
-      <limit effort="15.0" lower="${-PI}" upper="${PI}" velocity="30"/>
+      <limit effort="50.0" lower="${-PI}" upper="${PI}" velocity="30"/>
     </joint>
     <joint name="wheel_jointL" type="continuous">
@@ -188,6 +188,6 @@
       <origin rpy="0.0 0.0 0.0" xyz="0.1414 0.02 -0.1414"/>
       <axis xyz="0.0 1.0 0.0"/>
-      <dynamics damping="0.1" friction="0.05"/>
-      <limit effort="100.0" velocity="30"/>
+      <dynamics damping="0.1" friction="0.0"/>
+      <limit effort="300.0" velocity="3000"/>
     </joint>
     <!-- Right Side -->
@@ -296,5 +296,5 @@
       </collision>
     </link>
-    <joint name="hip_jointR" type="revolute">
+    <joint name="hip_jointR" type="fixed">
       <parent link="base_link"/>
       <child link="hip_motorR"/>
@@ -314,5 +314,5 @@
       <origin rpy="0.0 0.0 0.0" xyz="0.0 -0.035 0.0"/>
     </joint>
-    <joint name="knee_jointR" type="revolute">
+    <joint name="knee_jointR" type="fixed">
       <parent link="knee_motorR"/>
       <child link="knee_linkR"/>
@@ -322,5 +322,5 @@
       <limit effort="15.0" lower="${-PI}" upper="${PI}" velocity="30"/>
     </joint>
-    <joint name="virtualhip_jointR" type="revolute">
+    <joint name="virtualhip_jointR" type="fixed">
       <parent link="knee_linkR"/>
       <child link="leg_linkR"/>
@@ -335,6 +335,6 @@
       <origin rpy="0.0 0.0 0.0" xyz="0.1414 -0.02 -0.1414"/>
       <axis xyz="0.0 1.0 0.0"/>
-      <dynamics damping="0.1" friction="0.05"/>
-      <limit effort="100.0" velocity="30"/>
+      <dynamics damping="0.1" friction="0.0"/>
+      <limit effort="300.0" velocity="3000"/>
     </joint>
     <gazebo reference="imu_link">

Commit message: traj

File: otto_simulation/urdf/otto-simulationtest.xacro (robot description, xacro)
@@ -13,9 +13,9 @@
     <link name="base_link">
         <inertial>
-          <origin xyz="-0.025374 0.0 0.0" rpy="0 0 0"/>
-          <mass value="5.21707"/>
-          <inertia ixx="25.36345483e-3" ixy="0.0" ixz="-2.72079904e-3"
-                   iyx="0.0" iyy="28.97825187e-3" iyz="0.0"
-                   izx="-2.72079904e-3" izy="0.0" izz="35.16013094e-3" />
+          <origin xyz="-0.02195199 0.0 0.0" rpy="0 0 0"/>
+          <mass value="3.00"/>
+          <inertia ixx="14584893e-9" ixy="0.0" ixz="0.0"
+                   iyx="0.0" iyy="16663530e-9" iyz="0.0"
+                   izx="0.0" izy="0.0" izz="20218332e-9" />
         </inertial>
         <visual>
@@ -188,5 +188,5 @@
       <origin rpy="0.0 0.0 0.0" xyz="0.1414 0.02 -0.1414"/>
       <axis xyz="0.0 1.0 0.0"/>
-      <dynamics damping="0.1" friction="0.0"/>
+      <dynamics damping="0.01" friction="0.0"/>
       <limit effort="300.0" velocity="3000"/>
     </joint>
@@ -317,5 +317,5 @@
       <parent link="knee_motorR"/>
       <child link="knee_linkR"/>
-      <origin rpy="0.0 0.0 0.0" xyz="0.0 -0.05 0.0"/>
+      <origin rpy="0.0 0.0 0.0" xyz="0.0 -0.055 0.0"/>
       <axis xyz="0.0 1.0 0.0"/>
       <dynamics damping="0.1" friction="0.02"/>
@@ -335,5 +335,5 @@
       <origin rpy="0.0 0.0 0.0" xyz="0.1414 -0.02 -0.1414"/>
       <axis xyz="0.0 1.0 0.0"/>
-      <dynamics damping="0.1" friction="0.0"/>
+      <dynamics damping="0.01" friction="0.0"/>
       <limit effort="300.0" velocity="3000"/>
     </joint>
@@ -342,10 +342,10 @@
       <sensor name="imu_sensor" type="imu">
         <always_on>true</always_on>
-        <update_rate>1000</update_rate>
+        <update_rate>500.0</update_rate>
         <visualize>true</visualize>
         <plugin filename="libgazebo_ros_imu_sensor.so" name="imu_plugin">
           <topicName>otto_imu</topicName>
           <bodyName>imu_link</bodyName>
-          <updateRateHZ>1000.0</updateRateHZ>
+          <updateRateHZ>200.0</updateRateHZ>
           <gaussianNoise>0.0</gaussianNoise>
           <xyzOffset>0 0 0</xyzOffset>
