Commit message: lom dai laew

File: otto_simulation/urdf/gazebo.xacro (robot description, xacro)
@@ -1,4 +1,5 @@
 <?xml version="1.0"?>
 <robot xmlns:xacro="http://www.ros.org/wiki/xacro" name="otto">
+<!--
     <ros2_control name="GazeboSystem" type="system">
         <hardware>
@@ -69,5 +70,5 @@
             <state_interface name="effort"/>
         </joint>
-    </ros2_control>
+    </ros2_control> -->
     <gazebo>
         <plugin filename="libgazebo_ros2_control.so" name="gazebo_ros2_control">

File: otto_simulation/urdf/otto-simulation.xacro (robot description, xacro)
@@ -12,11 +12,11 @@
     <!-- Base Link -->
     <link name="base_link">
-        <!-- <inertial>
+        <inertial>
           <origin xyz="0.0 0.0 0.0" rpy="0 0 0"/>
           <mass value="5.21707"/>
-          <inertia ixx="25.36345483" ixy="0.0" ixz="-2.72079904"
-                   iyx="0.0" iyy="28.97825187" iyz="0.0"
-                   izx="-2.72079904" izy="0.0" izz="35.16013094" />
-        </inertial> -->
+          <inertia ixx="25.36345483e-3" ixy="0.0" ixz="-2.72079904e-3"
+                   iyx="0.0" iyy="28.97825187e-3" iyz="0.0"
+                   izx="-2.72079904e-3" izy="0.0" izz="35.16013094e-3" />
+        </inertial>
         <visual>
             <origin rpy="0.0 0.0 0.0" xyz="0.0 0.0 0.0"/>
@@ -37,7 +37,7 @@
         <origin xyz="0.0 0.0 0.0" rpy="0 0 0"/>
         <mass value="0.11255"/>
-        <inertia ixx="0.090104" ixy="0.000735" ixz="0.00035172"
-                 iyx="0.000735" iyy="0.074462" iyz="0.000140"
-                 izx="0.000351" izy="0.000140" izz="0.091432" />
+        <inertia ixx="0.090104e-3" ixy="0.000735e-3" ixz="0.00035172e-3"
+                 iyx="0.000735e-3" iyy="0.074462e-3" iyz="0.000140e-3"
+                 izx="0.000351e-3" izy="0.000140e-3" izz="0.091432e-3" />
       </inertial>
       <visual>
@@ -53,7 +53,7 @@
         <origin xyz="0.0 0.0 0.0" rpy="0 0 0"/>
         <mass value="0.11255"/>
-        <inertia ixx="0.090104" ixy="0.000735" ixz="0.00035172"
-                 iyx="0.000735" iyy="0.074462" iyz="0.000140"
-                 izx="0.000351" izy="0.000140" izz="0.091432" />
+        <inertia ixx="0.090104e-3" ixy="0.000735e-3" ixz="0.00035172e-3"
+                 iyx="0.000735e-3" iyy="0.074462e-3" iyz="0.000140e-3"
+                 izx="0.000351e-3" izy="0.000140e-3" izz="0.091432e-3" />
       </inertial>
       <visual>
@@ -69,7 +69,7 @@
         <origin xyz="0.0 0.0 0.0" rpy="0 0 0"/>
         <mass value="0.036"/>
-        <inertia ixx="0.038283" ixy="-0.00189" ixz="-0.020858"
-                 iyx="0.00189" iyy="0.066365" iyz="0.0021110"
-                 izx="0.0208580" izy="0.0021110" izz="0.030274" />
+        <inertia ixx="0.038283e-3" ixy="-0.00189e-3" ixz="-0.020858e-3"
+                 iyx="0.00189e-3" iyy="0.066365e-3" iyz="0.0021110e-3"
+                 izx="0.0208580e-3" izy="0.0021110e-3" izz="0.030274e-3" />
       </inertial>
       <visual>
@@ -84,8 +84,6 @@
       <inertial>
         <origin xyz="0.0 0.0 0.0" rpy="0 0 0"/>
-        <mass value="0.096"/>
-        <inertia ixx="0.808404" ixy="-0.054285" ixz="0.744011"
-                 iyx="-0.054285" iyy="1.51041728" iyz="-0.061449"
-                 izx="0.744011" izy="-0.061449" izz="0.743050" />
+        <mass value="0.09629"/>
+        <inertia ixx="808404e-10" iyy="1510417e-10" izz="743050e-10" ixy="0.0" iyz="0.0" ixz="0.0"/>
       </inertial>
       <visual>
@@ -101,7 +99,5 @@
         <origin xyz="0.0 0.0 0.0" rpy="0 0 0"/>
         <mass value="0.08537"/>
-        <inertia ixx="0.421600" ixy="0.022038" ixz="-0.474866"
-                 iyx="0.022038" iyy="0.982737" iyz="-0.017606"
-                 izx="-0.474866" izy="-0.017606" izz="0.566988" />
+        <inertia ixx="421600e-9" iyy="982737e-9" izz="566988e-9" ixy="0.0" iyz="0.0" ixz="0.0"/>
       </inertial>
       <visual>
@@ -117,7 +113,7 @@
         <origin xyz="0.0 0.0 0.0" rpy="0 0 0"/>
         <mass value="0.51691"/>
-        <inertia ixx="1.717624" ixy="0.000049" ixz="-0.000006"
-                 iyx="0.000049" iyy="2.388020" iyz="0.000004"
-                 izx="-0.000006" izy="-0.000015" izz="1.717603" />
+        <inertia ixx="1.717624e-3" ixy="0.000049e-3" ixz="-0.000006e-3"
+                 iyx="0.000049e-3" iyy="2.388020e-3" iyz="0.000004e-3"
+                 izx="-0.000006e-3" izy="-0.000015e-3" izz="1.717603e-3" />
       </inertial>
       <visual>
@@ -134,5 +130,5 @@
       </collision>
     </link>
-    <joint name="hip_jointL" type="continuous">
+    <joint name="hip_jointL" type="fixed">
       <parent link="base_link"/>
       <child link="hip_motorL"/>
@@ -151,5 +147,5 @@
       <origin rpy="0.0 0.0 0.0" xyz="0.0 0.035 0.0"/>
     </joint>
-    <joint name="knee_jointL" type="continuous">
+    <joint name="knee_jointL" type="fixed">
       <parent link="knee_motorL"/>
       <child link="knee_linkL"/>
@@ -158,5 +154,5 @@
       <dynamics damping="0.1" friction="0.05"/>
     </joint>
-    <joint name="virtualhip_jointL" type="continuous">
+    <joint name="virtualhip_jointL" type="fixed">
       <parent link="knee_linkL"/>
       <child link="leg_linkL"/>
@@ -165,5 +161,5 @@
       <dynamics damping="0.1" friction="0.05"/>
     </joint>
-    <joint name="wheel_jointL" type="continuous">
+    <joint name="wheel_jointL" type="fixed">
       <parent link="leg_linkL"/>
       <child link="wheel_linkL"/>
@@ -178,7 +174,7 @@
         <origin xyz="0.0 0.0 0.0" rpy="0 0 0"/>
         <mass value="0.11255"/>
-        <inertia ixx="0.090104" ixy="0.000735" ixz="0.00035172"
-                 iyx="0.000735" iyy="0.074462" iyz="0.000140"
-                 izx="0.000351" izy="0.000140" izz="0.091432" />
+        <inertia ixx="0.090104e-3" ixy="0.000735e-3" ixz="0.00035172e-3"
+                 iyx="0.000735e-3" iyy="0.074462e-3" iyz="0.000140e-3"
+                 izx="0.000351e-3" izy="0.000140e-3" izz="0.091432e-3" />
       </inertial>
       <visual>
@@ -193,8 +189,8 @@
       <inertial>
         <origin xyz="0.0 0.0 0.0" rpy="0 0 0"/>
-        <mass value="0.096"/>
-        <inertia ixx="0.808404" ixy="0.054285" ixz="0.744011"
-                 iyx="0.054285" iyy="1.51041728" iyz="0.061449"
-                 izx="0.744011" izy="0.061449" izz="0.743050" />
+        <mass value="0.11255"/>
+        <inertia ixx="0.090104e-3" ixy="0.000735e-3" ixz="0.00035172e-3"
+                 iyx="0.000735e-3" iyy="0.074462e-3" iyz="0.000140e-3"
+                 izx="0.000351e-3" izy="0.000140e-3" izz="0.091432e-3" />
       </inertial>
       <visual>
@@ -210,7 +206,7 @@
         <origin xyz="0.0 0.0 0.0" rpy="0 0 0"/>
         <mass value="0.036"/>
-        <inertia ixx="0.038283" ixy="0.00189" ixz="-0.020858"
-                 iyx="0.00189" iyy="0.066365" iyz="-0.0021110"
-                 izx="-0.0208580" izy="-0.0021110" izz="0.030274" />
+        <inertia ixx="0.038283e-3" ixy="0.00189e-3" ixz="-0.020858e-3"
+                 iyx="0.00189e-3" iyy="0.066365e-3" iyz="-0.0021110e-3"
+                 izx="-0.0208580e-3" izy="-0.0021110e-3" izz="0.030274e-3" />
       </inertial>
       <visual>
@@ -225,8 +221,6 @@
       <inertial>
         <origin xyz="0.0 0.0 0.0" rpy="0 0 0"/>
-        <mass value="0.096"/>
-        <inertia ixx="0.808404" ixy="0.054285" ixz="0.744011"
-                 iyx="0.054285" iyy="1.51041728" iyz="0.061449"
-                 izx="0.744011" izy="-0.061449" izz="0.743050" />
+        <mass value="0.09629"/>
+        <inertia ixx="808404e-10" iyy="1510417e-10" izz="743050e-10" ixy="0.0" iyz="0.0" ixz="0.0"/>
       </inertial>
       <visual>
@@ -242,7 +236,5 @@
         <origin xyz="0.0 0.0 0.0" rpy="0 0 0"/>
         <mass value="0.08537"/>
-        <inertia ixx="0.421600" ixy="-0.022038" ixz="-0.474866"
-                 iyx="-0.022038" iyy="0.982737" iyz="0.017606"
-                 izx="-0.474866" izy="0.017606" izz="0.566988" />
+        <inertia ixx="421600e-9" iyy="982737e-9" izz="566988e-9" ixy="0.0" iyz="0.0" ixz="0.0"/>
       </inertial>
       <visual>
@@ -258,7 +250,7 @@
         <origin xyz="0.0 0.0 0.0" rpy="0 0 0"/>
         <mass value="0.51691"/>
-        <inertia ixx="1.717624" ixy="0.000049" ixz="-0.000006"
-                 iyx="0.000049" iyy="2.388020" iyz="0.000004"
-                 izx="-0.000006" izy="-0.000015" izz="1.717603" />
+        <inertia ixx="1.717624e-3" ixy="0.000049e-3" ixz="-0.000006e-3"
+                 iyx="0.000049e-3" iyy="2.388020e-3" iyz="0.000004e-3"
+                 izx="-0.000006e-3" izy="-0.000015e-3" izz="1.717603e-3" />
       </inertial>
       <visual>
@@ -275,5 +267,5 @@
       </collision>
     </link>
-    <joint name="hip_jointR" type="continuous">
+    <joint name="hip_jointR" type="fixed">
       <parent link="base_link"/>
       <child link="hip_motorR"/>
@@ -285,5 +277,5 @@
       <parent link="hip_motorR"/>
       <child link="knee_motorR"/>
-        <origin rpy="0.0 0.0 0.0" xyz="0.0 -0.05 0.0"/>
+      <origin rpy="0.0 0.0 0.0" xyz="0.0 -0.05 0.0"/>
     </joint>
     <joint name="hip_motorR_to_hip_linkR" type="fixed">
@@ -292,5 +284,5 @@
       <origin rpy="0.0 0.0 0.0" xyz="0.0 -0.035 0.0"/>
     </joint>
-    <joint name="knee_jointR" type="continuous">
+    <joint name="knee_jointR" type="fixed">
       <parent link="knee_motorR"/>
       <child link="knee_linkR"/>
@@ -299,5 +291,5 @@
       <dynamics damping="0.1" friction="0.05"/>
     </joint>
-    <joint name="virtualhip_jointR" type="continuous">
+    <joint name="virtualhip_jointR" type="fixed">
       <parent link="knee_linkR"/>
       <child link="leg_linkR"/>
@@ -306,5 +298,5 @@
       <dynamics damping="0.1" friction="0.05"/>
     </joint>
-    <joint name="wheel_jointR" type="continuous">
+    <joint name="wheel_jointR" type="fixed">
       <parent link="leg_linkR"/>
       <child link="wheel_linkR"/>

Commit message: add transmission

File: otto_simulation/urdf/gazebo.xacro (robot description, xacro)
@@ -1,142 +1,152 @@
 <?xml version="1.0"?>
 <robot xmlns:xacro="http://www.ros.org/wiki/xacro" name="otto">
-<!--
-    <ros2_control name="GazeboSystem" type="system">
-        <hardware>
-            <plugin>gazebo_ros2_control/GazeboSystem</plugin>
-        </hardware>
-        <joint name="hip_jointL">
-            <command_interface name="position"/>
-            <state_interface name="position">
-                <param name="initial_value">0.0</param>
-            </state_interface>
-            <state_interface name="velocity"/>
-            <state_interface name="effort"/>
-        </joint>
-        <joint name="knee_jointL">
-            <command_interface name="position"/>
-            <state_interface name="position">
-                <param name="initial_value">0.0</param>
-            </state_interface>
-            <state_interface name="velocity"/>
-            <state_interface name="effort"/>
-        </joint>
-        <joint name="virtualhip_jointL">
-            <command_interface name="position"/>
-            <state_interface name="position">
-                <param name="initial_value">0.0</param>
-            </state_interface>
-            <state_interface name="velocity"/>
-            <state_interface name="effort"/>
-        </joint>
-        <joint name="wheel_jointL">
-            <command_interface name="position"/>
-            <state_interface name="position">
-                <param name="initial_value">0.0</param>
-            </state_interface>
-            <state_interface name="velocity"/>
-            <state_interface name="effort"/>
-        </joint>
-        <joint name="hip_jointR">
-            <command_interface name="position"/>
-            <state_interface name="position">
-                <param name="initial_value">0.0</param>
-            </state_interface>
-            <state_interface name="velocity"/>
-            <state_interface name="effort"/>
-        </joint>
-        <joint name="knee_jointR">
-            <command_interface name="position"/>
-            <state_interface name="position">
-                <param name="initial_value">0.0</param>
-            </state_interface>
-            <state_interface name="velocity"/>
-            <state_interface name="effort"/>
-        </joint>
-        <joint name="virtualhip_jointR">
-            <command_interface name="position"/>
-            <state_interface name="position">
-                <param name="initial_value">0.0</param>
-            </state_interface>
-            <state_interface name="velocity"/>
-            <state_interface name="effort"/>
-        </joint>
-        <joint name="wheel_jointR">
-            <command_interface name="position"/>
-            <state_interface name="position">
-                <param name="initial_value">0.0</param>
-            </state_interface>
-            <state_interface name="velocity"/>
-            <state_interface name="effort"/>
-        </joint>
-    </ros2_control> -->
+    <gazebo>
+        <plugin name="joint_state_publisher" filename="libgazebo_ros_joint_state_publisher.so">
+            <joint_name>hip_jointL</joint_name>
+            <joint_name>knee_jointL</joint_name>
+            <joint_name>virtualhip_jointL</joint_name>
+            <joint_name>wheel_jointL</joint_name>
+            <joint_name>hip_jointR</joint_name>
+            <joint_name>knee_jointR</joint_name>
+            <joint_name>virtualhip_jointR</joint_name>
+            <joint_name>wheel_jointR</joint_name>
+            <update_rate>30</update_rate>
+        </plugin>
+    </gazebo>
     <gazebo>
         <plugin filename="libgazebo_ros2_control.so" name="gazebo_ros2_control">
-            <robot_sim_type>gazebo_ros2_control/GazeboSystem</robot_sim_type>
-            <parameters>$(find otto_simulation)/config/joints_controller.yaml</parameters>
+            <!-- <parameters>$(find otto_simulation)/config/joints_controller.yaml</parameters> -->
         </plugin>
     </gazebo>
+    <transmission name="tran1">
+        <type>transmission_interface/SimpleTransmission</type>
+        <joint name="hip_jointL">
+          <hardwareInterface>hardware_interface/EffortJointInterface</hardwareInterface>
+        </joint>
+        <actuator name="actr1">
+          <hardwareInterface>hardware_interface/EffortJointInterface</hardwareInterface>
+          <mechanicalReduction>1</mechanicalReduction>
+        </actuator>
+    </transmission>
+    <transmission name="tran2">
+        <type>transmission_interface/SimpleTransmission</type>
+        <joint name="knee_jointL">
+          <hardwareInterface>hardware_interface/EffortJointInterface</hardwareInterface>
+        </joint>
+        <actuator name="actr2">
+          <hardwareInterface>hardware_interface/EffortJointInterface</hardwareInterface>
+          <mechanicalReduction>1</mechanicalReduction>
+        </actuator>
+    </transmission>
+    <transmission name="tran3">
+        <type>transmission_interface/SimpleTransmission</type>
+        <joint name="virtualhip_jointL">
+          <hardwareInterface>hardware_interface/EffortJointInterface</hardwareInterface>
+        </joint>
+        <actuator name="actr3">
+          <hardwareInterface>hardware_interface/EffortJointInterface</hardwareInterface>
+          <mechanicalReduction>1</mechanicalReduction>
+        </actuator>
+    </transmission>
+    <transmission name="tran4">
+        <type>transmission_interface/SimpleTransmission</type>
+        <joint name="wheel_jointL">
+          <hardwareInterface>hardware_interface/EffortJointInterface</hardwareInterface>
+        </joint>
+        <actuator name="actr4">
+          <hardwareInterface>hardware_interface/EffortJointInterface</hardwareInterface>
+          <mechanicalReduction>1</mechanicalReduction>
+        </actuator>
+    </transmission>
+    <transmission name="tran5">
+        <type>transmission_interface/SimpleTransmission</type>
+        <joint name="hip_jointR">
+          <hardwareInterface>hardware_interface/EffortJointInterface</hardwareInterface>
+        </joint>
+        <actuator name="actr5">
+          <hardwareInterface>hardware_interface/EffortJointInterface</hardwareInterface>
+          <mechanicalReduction>1</mechanicalReduction>
+        </actuator>
+    </transmission>
+    <transmission name="tran6">
+        <type>transmission_interface/SimpleTransmission</type>
+        <joint name="knee_jointR">
+          <hardwareInterface>hardware_interface/EffortJointInterface</hardwareInterface>
+        </joint>
+        <actuator name="actr6">
+          <hardwareInterface>hardware_interface/EffortJointInterface</hardwareInterface>
+          <mechanicalReduction>1</mechanicalReduction>
+        </actuator>
+    </transmission>
+    <transmission name="tran7">
+        <type>transmission_interface/SimpleTransmission</type>
+        <joint name="virtualhip_jointR">
+          <hardwareInterface>hardware_interface/EffortJointInterface</hardwareInterface>
+        </joint>
+        <actuator name="actr7">
+          <hardwareInterface>hardware_interface/EffortJointInterface</hardwareInterface>
+          <mechanicalReduction>1</mechanicalReduction>
+        </actuator>
+    </transmission>
+    <transmission name="tran8">
+        <type>transmission_interface/SimpleTransmission</type>
+        <joint name="wheel_jointR">
+          <hardwareInterface>hardware_interface/EffortJointInterface</hardwareInterface>
+        </joint>
+        <actuator name="actr8">
+          <hardwareInterface>hardware_interface/EffortJointInterface</hardwareInterface>
+          <mechanicalReduction>1</mechanicalReduction>
+        </actuator>
+    </transmission>
     <gazebo reference="base_link">
-        <mu1>0.2</mu1>
-        <mu2>0.2</mu2>
-        <material>Gazebo/Green</material>
+        <mu1>1.0</mu1>
+        <mu2>1.0</mu2>
+        <minDepth>0.0002</minDepth>
+        <kp  value="1000000.0"/>
+        <kd  value="100.0"/>
     </gazebo>
     <gazebo reference="hip_motorL">
-        <mu1>0.2</mu1>
-        <mu2>0.2</mu2>
         <material>Gazebo/Red</material>
     </gazebo>
     <gazebo reference="knee_motorL">
-        <mu1>0.2</mu1>
-        <mu2>0.2</mu2>
         <material>Gazebo/Blue</material>
     </gazebo>
     <gazebo reference="hip_linkL">
-        <mu1>0.2</mu1>
-        <mu2>0.2</mu2>
         <material>Gazebo/Black</material>
     </gazebo>
     <gazebo reference="knee_linkL">
-        <mu1>0.2</mu1>
-        <mu2>0.2</mu2>
         <material>Gazebo/Black</material>
     </gazebo>
     <gazebo reference="leg_linkL">
-        <mu1>0.2</mu1>
-        <mu2>0.2</mu2>
         <material>Gazebo/Black</material>
     </gazebo>
     <gazebo reference="wheel_linkL">
-        <mu1>0.2</mu1>
-        <mu2>0.2</mu2>
+        <mu1>1.0</mu1>
+        <mu2>1.0</mu2>
+        <minDepth>0.0002</minDepth>
+        <kp  value="1000000.0"/>
+        <kd  value="100.0"/>
     </gazebo>
     <gazebo reference="hip_motorR">
-        <mu1>0.2</mu1>
-        <mu2>0.2</mu2>
         <material>Gazebo/Red</material>
     </gazebo>
     <gazebo reference="knee_motorR">
-        <mu1>0.2</mu1>
-        <mu2>0.2</mu2>
         <material>Gazebo/Blue</material>
     </gazebo>
     <gazebo reference="hip_linkR">
-        <mu1>0.2</mu1>
-        <mu2>0.2</mu2>
         <material>Gazebo/Black</material>
     </gazebo>
     <gazebo reference="knee_linkR">
-        <mu1>0.2</mu1>
-        <mu2>0.2</mu2>
         <material>Gazebo/Black</material>
     </gazebo>
     <gazebo reference="leg_linkR">
-        <mu1>0.2</mu1>
-        <mu2>0.2</mu2>
         <material>Gazebo/Black</material>
     </gazebo>
     <gazebo reference="wheel_linkR">
-        <mu1>0.2</mu1>
-        <mu2>0.2</mu2>
+        <mu1>1.0</mu1>
+        <mu2>1.0</mu2>
+        <minDepth>0.0002</minDepth>
+        <kp  value="1000000.0"/>
+        <kd  value="100.0"/>
     </gazebo>
 </robot>

File: otto_simulation/urdf/otto-simulation.xacro (robot description, xacro)
@@ -130,5 +130,5 @@
       </collision>
     </link>
-    <joint name="hip_jointL" type="fixed">
+    <joint name="hip_jointL" type="continuous">
       <parent link="base_link"/>
       <child link="hip_motorL"/>
@@ -147,5 +147,5 @@
       <origin rpy="0.0 0.0 0.0" xyz="0.0 0.035 0.0"/>
     </joint>
-    <joint name="knee_jointL" type="fixed">
+    <joint name="knee_jointL" type="continuous">
       <parent link="knee_motorL"/>
       <child link="knee_linkL"/>
@@ -154,5 +154,5 @@
       <dynamics damping="0.1" friction="0.05"/>
     </joint>
-    <joint name="virtualhip_jointL" type="fixed">
+    <joint name="virtualhip_jointL" type="continuous">
       <parent link="knee_linkL"/>
       <child link="leg_linkL"/>
@@ -161,5 +161,5 @@
       <dynamics damping="0.1" friction="0.05"/>
     </joint>
-    <joint name="wheel_jointL" type="fixed">
+    <joint name="wheel_jointL" type="continuous">
       <parent link="leg_linkL"/>
       <child link="wheel_linkL"/>
@@ -267,5 +267,5 @@
       </collision>
     </link>
-    <joint name="hip_jointR" type="fixed">
+    <joint name="hip_jointR" type="continuous">
       <parent link="base_link"/>
       <child link="hip_motorR"/>
@@ -284,5 +284,5 @@
       <origin rpy="0.0 0.0 0.0" xyz="0.0 -0.035 0.0"/>
     </joint>
-    <joint name="knee_jointR" type="fixed">
+    <joint name="knee_jointR" type="continuous">
       <parent link="knee_motorR"/>
       <child link="knee_linkR"/>
@@ -291,5 +291,5 @@
       <dynamics damping="0.1" friction="0.05"/>
     </joint>
-    <joint name="virtualhip_jointR" type="fixed">
+    <joint name="virtualhip_jointR" type="continuous">
       <parent link="knee_linkR"/>
       <child link="leg_linkR"/>
@@ -298,5 +298,5 @@
       <dynamics damping="0.1" friction="0.05"/>
     </joint>
-    <joint name="wheel_jointR" type="fixed">
+    <joint name="wheel_jointR" type="continuous">
       <parent link="leg_linkR"/>
       <child link="wheel_linkR"/>
