Commit message: can work without controller

File: otto_simulation/urdf/gazebo.xacro (robot description, xacro)
@@ -1,17 +1,4 @@
 <?xml version="1.0"?>
 <robot xmlns:xacro="http://www.ros.org/wiki/xacro" name="otto">
-    <gazebo>
-        <plugin name="joint_state_publisher" filename="libgazebo_ros_joint_state_publisher.so">
-            <joint_name>hip_jointL</joint_name>
-            <joint_name>knee_jointL</joint_name>
-            <joint_name>virtualhip_jointL</joint_name>
-            <joint_name>wheel_jointL</joint_name>
-            <joint_name>hip_jointR</joint_name>
-            <joint_name>knee_jointR</joint_name>
-            <joint_name>virtualhip_jointR</joint_name>
-            <joint_name>wheel_jointR</joint_name>
-            <update_rate>30</update_rate>
-        </plugin>
-    </gazebo>
     <gazebo>
         <plugin filename="libgazebo_ros2_control.so" name="gazebo_ros2_control">
@@ -19,84 +6,105 @@
         </plugin>
     </gazebo>
-    <transmission name="tran1">
-        <type>transmission_interface/SimpleTransmission</type>
+    <!-- <ros2_control name="GazeboSystem" type="system">
+        <hardware>
+            <plugin>gazebo_ros2_control/GazeboSystem</plugin>
+        </hardware>
         <joint name="hip_jointL">
-          <hardwareInterface>hardware_interface/EffortJointInterface</hardwareInterface>
+            <param name="pos_kp">10</param>
+            <param name="pos_ki">1</param>
+            <param name="pos_kd">2</param>
+            <param name="pos_max_integral_error">10000</param>
+            <command_interface name="position_pid"/>
+            <state_interface name="position">
+              <param name="initial_value">0.0</param>
+            </state_interface>
+            <state_interface name="velocity"/>
+            <state_interface name="effort"/>
         </joint>
-        <actuator name="actr1">
-          <hardwareInterface>hardware_interface/EffortJointInterface</hardwareInterface>
-          <mechanicalReduction>1</mechanicalReduction>
-        </actuator>
-    </transmission>
-    <transmission name="tran2">
-        <type>transmission_interface/SimpleTransmission</type>
         <joint name="knee_jointL">
-          <hardwareInterface>hardware_interface/EffortJointInterface</hardwareInterface>
+            <param name="pos_kp">10</param>
+            <param name="pos_ki">1</param>
+            <param name="pos_kd">2</param>
+            <param name="pos_max_integral_error">10000</param>
+            <command_interface name="position_pid"/>
+            <state_interface name="position">
+              <param name="initial_value">0.0</param>
+            </state_interface>
+            <state_interface name="velocity"/>
+            <state_interface name="effort"/>
         </joint>
-        <actuator name="actr2">
-          <hardwareInterface>hardware_interface/EffortJointInterface</hardwareInterface>
-          <mechanicalReduction>1</mechanicalReduction>
-        </actuator>
-    </transmission>
-    <transmission name="tran3">
-        <type>transmission_interface/SimpleTransmission</type>
         <joint name="virtualhip_jointL">
-          <hardwareInterface>hardware_interface/EffortJointInterface</hardwareInterface>
+            <param name="pos_kp">10</param>
+            <param name="pos_ki">1</param>
+            <param name="pos_kd">2</param>
+            <param name="pos_max_integral_error">10000</param>
+            <command_interface name="position_pid"/>
+            <state_interface name="position">
+              <param name="initial_value">0.0</param>
+            </state_interface>
+            <state_interface name="velocity"/>
+            <state_interface name="effort"/>
         </joint>
-        <actuator name="actr3">
-          <hardwareInterface>hardware_interface/EffortJointInterface</hardwareInterface>
-          <mechanicalReduction>1</mechanicalReduction>
-        </actuator>
-    </transmission>
-    <transmission name="tran4">
-        <type>transmission_interface/SimpleTransmission</type>
         <joint name="wheel_jointL">
-          <hardwareInterface>hardware_interface/EffortJointInterface</hardwareInterface>
+            <param name="vel_kp">10</param>
+            <param name="vel_ki">5</param>
+            <param name="vel_kd">2</param>
+            <param name="vel_max_integral_error">10000</param>
+            <command_interface name="velocity_pid"/>
+            <state_interface name="position">
+              <param name="initial_value">0.0</param>
+            </state_interface>
+            <state_interface name="velocity"/>
+            <state_interface name="effort"/>
         </joint>
-        <actuator name="actr4">
-          <hardwareInterface>hardware_interface/EffortJointInterface</hardwareInterface>
-          <mechanicalReduction>1</mechanicalReduction>
-        </actuator>
-    </transmission>
-    <transmission name="tran5">
-        <type>transmission_interface/SimpleTransmission</type>
         <joint name="hip_jointR">
-          <hardwareInterface>hardware_interface/EffortJointInterface</hardwareInterface>
+            <param name="pos_kp">10</param>
+            <param name="pos_ki">1</param>
+            <param name="pos_kd">2</param>
+            <param name="pos_max_integral_error">10000</param>
+            <command_interface name="position_pid"/>
+            <state_interface name="position">
+              <param name="initial_value">0.0</param>
+            </state_interface>
+            <state_interface name="velocity"/>
+            <state_interface name="effort"/>
         </joint>
-        <actuator name="actr5">
-          <hardwareInterface>hardware_interface/EffortJointInterface</hardwareInterface>
-          <mechanicalReduction>1</mechanicalReduction>
-        </actuator>
-    </transmission>
-    <transmission name="tran6">
-        <type>transmission_interface/SimpleTransmission</type>
         <joint name="knee_jointR">
-          <hardwareInterface>hardware_interface/EffortJointInterface</hardwareInterface>
+            <param name="pos_kp">10</param>
+            <param name="pos_ki">1</param>
+            <param name="pos_kd">2</param>
+            <param name="pos_max_integral_error">10000</param>
+            <command_interface name="position_pid"/>
+            <state_interface name="position">
+              <param name="initial_value">0.0</param>
+            </state_interface>
+            <state_interface name="velocity"/>
+            <state_interface name="effort"/>
         </joint>
-        <actuator name="actr6">
-          <hardwareInterface>hardware_interface/EffortJointInterface</hardwareInterface>
-          <mechanicalReduction>1</mechanicalReduction>
-        </actuator>
-    </transmission>
-    <transmission name="tran7">
-        <type>transmission_interface/SimpleTransmission</type>
         <joint name="virtualhip_jointR">
-          <hardwareInterface>hardware_interface/EffortJointInterface</hardwareInterface>
+            <param name="pos_kp">10</param>
+            <param name="pos_ki">1</param>
+            <param name="pos_kd">2</param>
+            <param name="pos_max_integral_error">10000</param>
+            <command_interface name="position_pid"/>
+            <state_interface name="position">
+              <param name="initial_value">0.0</param>
+            </state_interface>
+            <state_interface name="velocity"/>
+            <state_interface name="effort"/>
         </joint>
-        <actuator name="actr7">
-          <hardwareInterface>hardware_interface/EffortJointInterface</hardwareInterface>
-          <mechanicalReduction>1</mechanicalReduction>
-        </actuator>
-    </transmission>
-    <transmission name="tran8">
-        <type>transmission_interface/SimpleTransmission</type>
         <joint name="wheel_jointR">
-          <hardwareInterface>hardware_interface/EffortJointInterface</hardwareInterface>
+            <param name="vel_kp">10</param>
+            <param name="vel_ki">5</param>
+            <param name="vel_kd">2</param>
+            <param name="vel_max_integral_error">10000</param>
+            <command_interface name="velocity_pid"/>
+            <state_interface name="position">
+              <param name="initial_value">0.0</param>
+            </state_interface>
+            <state_interface name="velocity"/>
+            <state_interface name="effort"/>
         </joint>
-        <actuator name="actr8">
-          <hardwareInterface>hardware_interface/EffortJointInterface</hardwareInterface>
-          <mechanicalReduction>1</mechanicalReduction>
-        </actuator>
-    </transmission>
+    </ros2_control> -->
     <gazebo reference="base_link">
         <mu1>1.0</mu1>
@@ -105,4 +113,5 @@
         <kp  value="1000000.0"/>
         <kd  value="100.0"/>
+        <material>Gazebo/Green</material>
     </gazebo>
     <gazebo reference="hip_motorL">

File: otto_simulation/urdf/otto-simulation.xacro (robot description, xacro)
@@ -4,10 +4,10 @@
     <xacro:property name="PI" value="3.14159265359"/>
     <xacro:include filename="gazebo.xacro"/>
-    <!-- <link name="world"></link>
+    <link name="world"></link>
     <joint name="base_joint" type="fixed">
-      <origin xyz="0 0 0.0" rpy="0 0 0"/>
+      <origin xyz="0 0 0.3" rpy="0 0 0"/>
       <parent link="world"/>
       <child link="base_link"/>
-    </joint> -->
+    </joint>
     <!-- Base Link -->
     <link name="base_link">

Commit message: efffort controller

File: otto_simulation/urdf/gazebo.xacro (robot description, xacro)
@@ -6,105 +6,97 @@
         </plugin>
     </gazebo>
-    <!-- <ros2_control name="GazeboSystem" type="system">
+    <ros2_control name="GazeboSystem" type="system">
         <hardware>
             <plugin>gazebo_ros2_control/GazeboSystem</plugin>
         </hardware>
         <joint name="hip_jointL">
-            <param name="pos_kp">10</param>
-            <param name="pos_ki">1</param>
-            <param name="pos_kd">2</param>
-            <param name="pos_max_integral_error">10000</param>
-            <command_interface name="position_pid"/>
-            <state_interface name="position">
-              <param name="initial_value">0.0</param>
-            </state_interface>
-            <state_interface name="velocity"/>
-            <state_interface name="effort"/>
+            <command_interface name="effort">
+                <param name="min">-10000</param>
+                <param name="max">10000</param>
+              </command_interface>
+              <state_interface name="position">
+                <param name="initial_value">0.0</param>
+              </state_interface>
+              <state_interface name="velocity"/>
+              <state_interface name="effort"/>
         </joint>
         <joint name="knee_jointL">
-            <param name="pos_kp">10</param>
-            <param name="pos_ki">1</param>
-            <param name="pos_kd">2</param>
-            <param name="pos_max_integral_error">10000</param>
-            <command_interface name="position_pid"/>
-            <state_interface name="position">
-              <param name="initial_value">0.0</param>
-            </state_interface>
-            <state_interface name="velocity"/>
-            <state_interface name="effort"/>
+            <command_interface name="effort">
+                <param name="min">-10000</param>
+                <param name="max">10000</param>
+              </command_interface>
+              <state_interface name="position">
+                <param name="initial_value">0.0</param>
+              </state_interface>
+              <state_interface name="velocity"/>
+              <state_interface name="effort"/>
         </joint>
         <joint name="virtualhip_jointL">
-            <param name="pos_kp">10</param>
-            <param name="pos_ki">1</param>
-            <param name="pos_kd">2</param>
-            <param name="pos_max_integral_error">10000</param>
-            <command_interface name="position_pid"/>
-            <state_interface name="position">
-              <param name="initial_value">0.0</param>
-            </state_interface>
-            <state_interface name="velocity"/>
-            <state_interface name="effort"/>
+            <command_interface name="effort">
+                <param name="min">-10000</param>
+                <param name="max">10000</param>
+              </command_interface>
+              <state_interface name="position">
+                <param name="initial_value">0.0</param>
+              </state_interface>
+              <state_interface name="velocity"/>
+              <state_interface name="effort"/>
         </joint>
         <joint name="wheel_jointL">
-            <param name="vel_kp">10</param>
-            <param name="vel_ki">5</param>
-            <param name="vel_kd">2</param>
-            <param name="vel_max_integral_error">10000</param>
-            <command_interface name="velocity_pid"/>
-            <state_interface name="position">
-              <param name="initial_value">0.0</param>
-            </state_interface>
-            <state_interface name="velocity"/>
-            <state_interface name="effort"/>
+            <command_interface name="effort">
+                <param name="min">-10000</param>
+                <param name="max">10000</param>
+              </command_interface>
+              <state_interface name="position">
+                <param name="initial_value">0.0</param>
+              </state_interface>
+              <state_interface name="velocity"/>
+              <state_interface name="effort"/>
         </joint>
         <joint name="hip_jointR">
-            <param name="pos_kp">10</param>
-            <param name="pos_ki">1</param>
-            <param name="pos_kd">2</param>
-            <param name="pos_max_integral_error">10000</param>
-            <command_interface name="position_pid"/>
-            <state_interface name="position">
-              <param name="initial_value">0.0</param>
-            </state_interface>
-            <state_interface name="velocity"/>
-            <state_interface name="effort"/>
+            <command_interface name="effort">
+                <param name="min">-10000</param>
+                <param name="max">10000</param>
+              </command_interface>
+              <state_interface name="position">
+                <param name="initial_value">0.0</param>
+              </state_interface>
+              <state_interface name="velocity"/>
+              <state_interface name="effort"/>
         </joint>
         <joint name="knee_jointR">
-            <param name="pos_kp">10</param>
-            <param name="pos_ki">1</param>
-            <param name="pos_kd">2</param>
-            <param name="pos_max_integral_error">10000</param>
-            <command_interface name="position_pid"/>
-            <state_interface name="position">
-              <param name="initial_value">0.0</param>
-            </state_interface>
-            <state_interface name="velocity"/>
-            <state_interface name="effort"/>
+            <command_interface name="effort">
+                <param name="min">-10000</param>
+                <param name="max">10000</param>
+              </command_interface>
+              <state_interface name="position">
+                <param name="initial_value">0.0</param>
+              </state_interface>
+              <state_interface name="velocity"/>
+              <state_interface name="effort"/>
         </joint>
         <joint name="virtualhip_jointR">
-            <param name="pos_kp">10</param>
-            <param name="pos_ki">1</param>
-            <param name="pos_kd">2</param>
-            <param name="pos_max_integral_error">10000</param>
-            <command_interface name="position_pid"/>
-            <state_interface name="position">
-              <param name="initial_value">0.0</param>
-            </state_interface>
-            <state_interface name="velocity"/>
-            <state_interface name="effort"/>
+            <command_interface name="effort">
+                <param name="min">-10000</param>
+                <param name="max">10000</param>
+              </command_interface>
+              <state_interface name="position">
+                <param name="initial_value">0.0</param>
+              </state_interface>
+              <state_interface name="velocity"/>
+              <state_interface name="effort"/>
         </joint>
         <joint name="wheel_jointR">
-            <param name="vel_kp">10</param>
-            <param name="vel_ki">5</param>
-            <param name="vel_kd">2</param>
-            <param name="vel_max_integral_error">10000</param>
-            <command_interface name="velocity_pid"/>
-            <state_interface name="position">
-              <param name="initial_value">0.0</param>
-            </state_interface>
-            <state_interface name="velocity"/>
-            <state_interface name="effort"/>
+            <command_interface name="effort">
+                <param name="min">-10000</param>
+                <param name="max">10000</param>
+              </command_interface>
+              <state_interface name="position">
+                <param name="initial_value">0.0</param>
+              </state_interface>
+              <state_interface name="velocity"/>
+              <state_interface name="effort"/>
         </joint>
-    </ros2_control> -->
+    </ros2_control>
     <gazebo reference="base_link">
         <mu1>1.0</mu1>

File: otto_simulation/urdf/otto-simulation.xacro (robot description, xacro)
@@ -136,4 +136,5 @@
         <axis xyz="0.0 1.0 0.0"/>
       <dynamics damping="0.1" friction="0.05"/>
+      <limit effort="1000.0" lower="${PI}" upper="${-PI}" velocity="30"/>
     </joint>
     <joint name="hip_motorL_to_knee_motorL" type="fixed">
@@ -153,4 +154,5 @@
       <axis xyz="0.0 1.0 0.0"/>
       <dynamics damping="0.1" friction="0.05"/>
+      <limit effort="1000.0" lower="${PI}" upper="${-PI}" velocity="30"/>
     </joint>
     <joint name="virtualhip_jointL" type="continuous">
@@ -160,4 +162,5 @@
       <axis xyz="0.0 1.0 0.0"/>
       <dynamics damping="0.1" friction="0.05"/>
+      <limit effort="1000.0" lower="${PI}" upper="${-PI}" velocity="30"/>
     </joint>
     <joint name="wheel_jointL" type="continuous">
@@ -167,4 +170,5 @@
       <axis xyz="0.0 1.0 0.0"/>
       <dynamics damping="0.1" friction="0.05"/>
+      <limit effort="1000.0" velocity="30"/>
     </joint>
     <!-- Right Side -->
@@ -273,4 +277,5 @@
         <axis xyz="0.0 1.0 0.0"/>
         <dynamics damping="0.1" friction="0.05"/>
+        <limit effort="1000.0" lower="${PI}" upper="${-PI}" velocity="30"/>
     </joint>
     <joint name="hip_motorR_to_knee_motorR" type="fixed">
@@ -290,4 +295,5 @@
       <axis xyz="0.0 1.0 0.0"/>
       <dynamics damping="0.1" friction="0.05"/>
+      <limit effort="1000.0" lower="${PI}" upper="${-PI}" velocity="30"/>
     </joint>
     <joint name="virtualhip_jointR" type="continuous">
@@ -297,4 +303,5 @@
       <axis xyz="0.0 1.0 0.0"/>
       <dynamics damping="0.1" friction="0.05"/>
+      <limit effort="1000.0" lower="${PI}" upper="${-PI}" velocity="30"/>
     </joint>
     <joint name="wheel_jointR" type="continuous">
@@ -304,4 +311,5 @@
       <axis xyz="0.0 1.0 0.0"/>
       <dynamics damping="0.1" friction="0.05"/>
+      <limit effort="1000.0" velocity="30"/>
     </joint>
 </robot>
