Commit message: launch fix

File: otto_simulation/urdf/gazebo.xacro (robot description, xacro)
@@ -100,6 +100,4 @@
     </ros2_control>
     <gazebo reference="base_link">
-        <mu1>1.0</mu1>
-        <mu2>1.0</mu2>
         <minDepth>0.0002</minDepth>
         <kp  value="1000000.0"/>

File: otto_simulation/urdf/otto-simulation.xacro (robot description, xacro)
@@ -4,10 +4,10 @@
     <xacro:property name="PI" value="3.14159265359"/>
     <xacro:include filename="gazebo.xacro"/>
-    <link name="world"></link>
+    <!-- <link name="world"></link>
     <joint name="base_joint" type="fixed">
       <origin xyz="0.0 0.0 0.5" rpy="0.0 0.0 0.0"/>
       <parent link="world"/>
       <child link="base_link"/>
-    </joint>
+    </joint> -->
     <!-- Base Link -->
     <link name="base_link">
@@ -28,5 +28,5 @@
             <origin rpy="0.0 0.0 0.0" xyz="0.0 0.0 0.0"/>
             <geometry>
-                <box size="0.20 0.19 0.15"/>
+                <box size="0.22 0.19 0.15"/>
             </geometry>
         </collision>
@@ -107,4 +107,10 @@
           </geometry>
       </visual>
+      <collision>
+        <origin rpy="0.0 0.0 0.0" xyz="-0.05656 0.00 0.05656"/>
+        <geometry>
+            <sphere radius="0.01"/>
+        </geometry>
+      </collision>
     </link>
     <!-- wheel link Left -->
@@ -130,10 +136,10 @@
       </collision>
     </link>
-    <joint name="hip_jointL" type="continuous">
+    <joint name="hip_jointL" type="revolute">
       <parent link="base_link"/>
       <child link="hip_motorL"/>
         <origin rpy="0.0 0.0 0.0" xyz="-0.03 0.06 0.0"/>
         <axis xyz="0.0 1.0 0.0"/>
-      <dynamics damping="0.1" friction="0.05"/>
+      <dynamics damping="0.2" friction="0.05"/>
       <limit effort="100.0" lower="${PI}" upper="${-PI}" velocity="30"/>
     </joint>
@@ -148,13 +154,13 @@
       <origin rpy="0.0 0.0 0.0" xyz="0.0 0.035 0.0"/>
     </joint>
-    <joint name="knee_jointL" type="continuous">
+    <joint name="knee_jointL" type="revolute">
       <parent link="knee_motorL"/>
       <child link="knee_linkL"/>
       <origin rpy="0.0 0.0 0.0" xyz="0.0 0.055 0.0"/>
       <axis xyz="0.0 1.0 0.0"/>
-      <dynamics damping="0.1" friction="0.05"/>
-      <limit effort="100.0" lower="${PI}" upper="${-PI}" velocity="30"/>
-    </joint>
-    <joint name="virtualhip_jointL" type="continuous">
+      <dynamics damping="0.1" friction="0.02"/>
+      <limit effort="100.0" lower="${PI}" upper="${-PI}" velocity="30"/>
+    </joint>
+    <joint name="virtualhip_jointL" type="revolute">
       <parent link="knee_linkL"/>
       <child link="leg_linkL"/>
@@ -248,4 +254,10 @@
           </geometry>
       </visual>
+      <collision>
+        <origin rpy="0.0 0.0 0.0" xyz="-0.05656 0.00 0.05656"/>
+        <geometry>
+            <sphere radius="0.01"/>
+        </geometry>
+      </collision>
     </link>
     <!-- wheel link Right -->
@@ -271,10 +283,10 @@
       </collision>
     </link>
-    <joint name="hip_jointR" type="continuous">
+    <joint name="hip_jointR" type="revolute">
       <parent link="base_link"/>
       <child link="hip_motorR"/>
         <origin rpy="0.0 0.0 0.0" xyz="-0.03 -0.06 0.0"/>
         <axis xyz="0.0 1.0 0.0"/>
-        <dynamics damping="0.1" friction="0.05"/>
+        <dynamics damping="0.2" friction="0.05"/>
         <limit effort="100.0" lower="${PI}" upper="${-PI}" velocity="30"/>
     </joint>
@@ -289,13 +301,13 @@
       <origin rpy="0.0 0.0 0.0" xyz="0.0 -0.035 0.0"/>
     </joint>
-    <joint name="knee_jointR" type="continuous">
+    <joint name="knee_jointR" type="revolute">
       <parent link="knee_motorR"/>
       <child link="knee_linkR"/>
       <origin rpy="0.0 0.0 0.0" xyz="0.0 -0.05 0.0"/>
       <axis xyz="0.0 1.0 0.0"/>
-      <dynamics damping="0.1" friction="0.05"/>
-      <limit effort="100.0" lower="${PI}" upper="${-PI}" velocity="30"/>
-    </joint>
-    <joint name="virtualhip_jointR" type="continuous">
+      <dynamics damping="0.1" friction="0.02"/>
+      <limit effort="100.0" lower="${PI}" upper="${-PI}" velocity="30"/>
+    </joint>
+    <joint name="virtualhip_jointR" type="revolute">
       <parent link="knee_linkR"/>
       <child link="leg_linkR"/>

Commit message: not stable

File: otto_simulation/urdf/gazebo.xacro (robot description, xacro)
@@ -10,5 +10,5 @@
             <plugin>gazebo_ros2_control/GazeboSystem</plugin>
         </hardware>
-        <joint name="hip_jointL">
+        <!-- <joint name="hip_jointL">
             <command_interface name="effort">
                 <param name="min">-10000</param>
@@ -20,5 +20,5 @@
               <state_interface name="velocity"/>
               <state_interface name="effort"/>
-        </joint>
+        </joint> -->
         <joint name="knee_jointL">
             <command_interface name="effort">
@@ -54,5 +54,5 @@
               <state_interface name="effort"/>
         </joint>
-        <joint name="hip_jointR">
+        <!-- <joint name="hip_jointR">
             <command_interface name="effort">
                 <param name="min">-10000</param>
@@ -64,5 +64,5 @@
               <state_interface name="velocity"/>
               <state_interface name="effort"/>
-        </joint>
+        </joint> -->
         <joint name="knee_jointR">
             <command_interface name="effort">

File: otto_simulation/urdf/otto-simulation.xacro (robot description, xacro)
@@ -13,9 +13,9 @@
     <link name="base_link">
         <inertial>
-          <origin xyz="0.0 0.0 0.0" rpy="0 0 0"/>
-          <mass value="5.217065"/>
-          <inertia ixx="25.36345483e-3" ixy="0.0" ixz="-2.72079904e-3"
-                   iyx="0.0" iyy="28.97825187e-3" iyz="0.0"
-                   izx="-2.72079904e-3" izy="0.0" izz="35.16013094e-3" />
+          <origin xyz="-0.02195199 0.0 0.0" rpy="0 0 0"/>
+          <mass value="3.00"/>
+          <inertia ixx="14584893e-9" ixy="0.0" ixz="0.0"
+                   iyx="0.0" iyy="16663530e-9" iyz="0.0"
+                   izx="0.0" izy="0.0" izz="20218332e-9" />
         </inertial>
         <visual>
@@ -149,11 +149,10 @@
       </collision>
     </link>
-    <joint name="hip_jointL" type="revolute">
+    <joint name="hip_jointL" type="fixed">
       <parent link="base_link"/>
       <child link="hip_motorL"/>
         <origin rpy="0.0 0.0 0.0" xyz="-0.03 0.06 0.0"/>
         <axis xyz="0.0 1.0 0.0"/>
-      <dynamics damping="0.2" friction="0.05"/>
-      <limit effort="15.0" lower="${-PI}" upper="${PI}" velocity="30"/>
+        <!-- <limit effort="50.0" lower="${-PI}" upper="${PI}" velocity="30"/> -->
     </joint>
     <joint name="hip_motorL_to_knee_motorL" type="fixed">
@@ -167,19 +166,19 @@
       <origin rpy="0.0 0.0 0.0" xyz="0.0 0.035 0.0"/>
     </joint>
-    <joint name="knee_jointL" type="revolute">
+    <joint name="knee_jointL" type="continuous">
       <parent link="knee_motorL"/>
       <child link="knee_linkL"/>
       <origin rpy="0.0 0.0 0.0" xyz="0.0 0.055 0.0"/>
       <axis xyz="0.0 1.0 0.0"/>
-      <dynamics damping="0.1" friction="0.02"/>
-      <limit effort="15.0" lower="${-PI}" upper="${PI}" velocity="30"/>
-    </joint>
-    <joint name="virtualhip_jointL" type="revolute">
+      <dynamics damping="0.1" friction="0.0"/>
+      <!-- <limit effort="50.0" lower="${-PI}" upper="${PI}" velocity="30"/> -->
+    </joint>
+    <joint name="virtualhip_jointL" type="continuous">
       <parent link="knee_linkL"/>
       <child link="leg_linkL"/>
       <origin rpy="0.0 0.0 0.0" xyz="-0.1414 -0.05 -0.1414"/>
       <axis xyz="0.0 1.0 0.0"/>
-      <dynamics damping="0.1" friction="0.05"/>
-      <limit effort="15.0" lower="${-PI}" upper="${PI}" velocity="30"/>
+      <dynamics damping="0.1" friction="0.0"/>
+      <!-- <limit effort="50.0" lower="${-PI}" upper="${PI}" velocity="30"/> -->
     </joint>
     <joint name="wheel_jointL" type="continuous">
@@ -188,6 +187,6 @@
       <origin rpy="0.0 0.0 0.0" xyz="0.1414 0.02 -0.1414"/>
       <axis xyz="0.0 1.0 0.0"/>
-      <dynamics damping="0.1" friction="0.05"/>
-      <limit effort="100.0" velocity="30"/>
+      <dynamics damping="0.001" friction="0.0"/>
+      <limit effort="300.0" velocity="3000"/>
     </joint>
     <!-- Right Side -->
@@ -296,11 +295,10 @@
       </collision>
     </link>
-    <joint name="hip_jointR" type="revolute">
+    <joint name="hip_jointR" type="fixed">
       <parent link="base_link"/>
       <child link="hip_motorR"/>
         <origin rpy="0.0 0.0 0.0" xyz="-0.03 -0.06 0.0"/>
         <axis xyz="0.0 1.0 0.0"/>
-        <dynamics damping="0.2" friction="0.05"/>
-        <limit effort="15.0" lower="${-PI}" upper="${PI}" velocity="30"/>
+        <!-- <limit effort="15.0" lower="${-PI}" upper="${PI}" velocity="30"/> -->
       </joint>
     <joint name="hip_motorR_to_knee_motorR" type="fixed">
@@ -314,19 +312,19 @@
       <origin rpy="0.0 0.0 0.0" xyz="0.0 -0.035 0.0"/>
     </joint>
-    <joint name="knee_jointR" type="revolute">
+    <joint name="knee_jointR" type="continuous">
       <parent link="knee_motorR"/>
       <child link="knee_linkR"/>
-      <origin rpy="0.0 0.0 0.0" xyz="0.0 -0.05 0.0"/>
-      <axis xyz="0.0 1.0 0.0"/>
-      <dynamics damping="0.1" friction="0.02"/>
-      <limit effort="15.0" lower="${-PI}" upper="${PI}" velocity="30"/>
-    </joint>
-    <joint name="virtualhip_jointR" type="revolute">
+      <origin rpy="0.0 0.0 0.0" xyz="0.0 -0.055 0.0"/>
+      <axis xyz="0.0 1.0 0.0"/>
+      <dynamics damping="0.1" friction="0.0"/>
+      <!-- <limit effort="15.0" lower="${-PI}" upper="${PI}" velocity="30"/> -->
+    </joint>
+    <joint name="virtualhip_jointR" type="continuous">
       <parent link="knee_linkR"/>
       <child link="leg_linkR"/>
       <origin rpy="0.0 0.0 0.0" xyz="-0.1414 0.05 -0.1414"/>
       <axis xyz="0.0 1.0 0.0"/>
-      <dynamics damping="0.1" friction="0.05"/>
-      <limit effort="15.0" lower="${-PI}" upper="${PI}" velocity="30"/>
+      <dynamics damping="0.1" friction="0.0"/>
+      <!-- <limit effort="15.0" lower="${-PI}" upper="${PI}" velocity="30"/> -->
     </joint>
     <joint name="wheel_jointR" type="continuous">
@@ -335,6 +333,6 @@
       <origin rpy="0.0 0.0 0.0" xyz="0.1414 -0.02 -0.1414"/>
       <axis xyz="0.0 1.0 0.0"/>
-      <dynamics damping="0.1" friction="0.05"/>
-      <limit effort="100.0" velocity="30"/>
+      <dynamics damping="0.001" friction="0.0"/>
+      <limit effort="300.0" velocity="3000"/>
     </joint>
     <gazebo reference="imu_link">
@@ -342,10 +340,10 @@
       <sensor name="imu_sensor" type="imu">
         <always_on>true</always_on>
-        <update_rate>1000</update_rate>
+        <update_rate>500.0</update_rate>
         <visualize>true</visualize>
         <plugin filename="libgazebo_ros_imu_sensor.so" name="imu_plugin">
           <topicName>otto_imu</topicName>
           <bodyName>imu_link</bodyName>
-          <updateRateHZ>1000.0</updateRateHZ>
+          <updateRateHZ>200.0</updateRateHZ>
           <gaussianNoise>0.0</gaussianNoise>
           <xyzOffset>0 0 0</xyzOffset>

Commit message: stand up

File: otto_simulation/urdf/gazebo.xacro (robot description, xacro)
@@ -22,8 +22,13 @@
         </joint> -->
         <joint name="knee_jointL">
-            <command_interface name="effort">
+            <!-- <command_interface name="effort">
                 <param name="min">-10000</param>
                 <param name="max">10000</param>
-              </command_interface>
+              </command_interface> -->
+              <param name="pos_kp">100</param>
+              <param name="pos_ki">1</param>
+              <param name="pos_kd">10</param>
+              <param name="pos_max_integral_error">10000</param>
+              <command_interface name="position_pid"/>
               <state_interface name="position">
                 <param name="initial_value">0.0</param>
@@ -33,8 +38,9 @@
         </joint>
         <joint name="virtualhip_jointL">
-            <command_interface name="effort">
-                <param name="min">-10000</param>
-                <param name="max">10000</param>
-              </command_interface>
+              <param name="pos_kp">100</param>
+              <param name="pos_ki">1</param>
+              <param name="pos_kd">10</param>
+              <param name="pos_max_integral_error">10000</param>
+              <command_interface name="position_pid"/>
               <state_interface name="position">
                 <param name="initial_value">0.0</param>
@@ -66,8 +72,9 @@
         </joint> -->
         <joint name="knee_jointR">
-            <command_interface name="effort">
-                <param name="min">-10000</param>
-                <param name="max">10000</param>
-              </command_interface>
+              <param name="pos_kp">100</param>
+              <param name="pos_ki">1</param>
+              <param name="pos_kd">10</param>
+              <param name="pos_max_integral_error">10000</param>
+              <command_interface name="position_pid"/>
               <state_interface name="position">
                 <param name="initial_value">0.0</param>
@@ -77,8 +84,9 @@
         </joint>
         <joint name="virtualhip_jointR">
-            <command_interface name="effort">
-                <param name="min">-10000</param>
-                <param name="max">10000</param>
-              </command_interface>
+              <param name="pos_kp">100</param>
+              <param name="pos_ki">1</param>
+              <param name="pos_kd">10</param>
+              <param name="pos_max_integral_error">10000</param>
+              <command_interface name="position_pid"/>
               <state_interface name="position">
                 <param name="initial_value">0.0</param>

File: otto_simulation/urdf/otto-simulation.xacro (robot description, xacro)
@@ -98,5 +98,5 @@
         <origin xyz="0.0 0.0 0.0" rpy="0 0 0"/>
         <mass value="0.09629"/>
-        <inertia ixx="808404e-10" iyy="1510417e-10" izz="743050e-10" ixy="0.0" iyz="0.0" ixz="0.0"/>
+        <inertia ixx="808404e-9" iyy="1510417e-9" izz="743050e-9" ixy="0.0" iyz="0.0" ixz="0.0"/>
       </inertial>
       <visual>
@@ -172,5 +172,5 @@
       <axis xyz="0.0 1.0 0.0"/>
       <dynamics damping="0.1" friction="0.0"/>
-      <!-- <limit effort="50.0" lower="${-PI}" upper="${PI}" velocity="30"/> -->
+      <limit effort="5.5" lower="${-PI}" upper="${PI}" velocity="30"/>
     </joint>
     <joint name="virtualhip_jointL" type="continuous">
@@ -180,5 +180,5 @@
       <axis xyz="0.0 1.0 0.0"/>
       <dynamics damping="0.1" friction="0.0"/>
-      <!-- <limit effort="50.0" lower="${-PI}" upper="${PI}" velocity="30"/> -->
+      <limit effort="5.5" lower="${-PI}" upper="${PI}" velocity="30"/>
     </joint>
     <joint name="wheel_jointL" type="continuous">
@@ -188,5 +188,5 @@
       <axis xyz="0.0 1.0 0.0"/>
       <dynamics damping="0.001" friction="0.0"/>
-      <limit effort="300.0" velocity="3000"/>
+      <limit effort="300.0" velocity="50"/>
     </joint>
     <!-- Right Side -->
@@ -244,5 +244,5 @@
         <origin xyz="0.0 0.0 0.0" rpy="0 0 0"/>
         <mass value="0.09629"/>
-        <inertia ixx="808404e-10" iyy="1510417e-10" izz="743050e-10" ixy="0.0" iyz="0.0" ixz="0.0"/>
+        <inertia ixx="808404e-9" iyy="1510417e-9" izz="743050e-9" ixy="0.0" iyz="0.0" ixz="0.0"/>
       </inertial>
       <visual>
@@ -300,5 +300,5 @@
         <origin rpy="0.0 0.0 0.0" xyz="-0.03 -0.06 0.0"/>
         <axis xyz="0.0 1.0 0.0"/>
-        <!-- <limit effort="15.0" lower="${-PI}" upper="${PI}" velocity="30"/> -->
+        <!-- <limit effort="5.0" lower="${-PI}" upper="${PI}" velocity="30"/> -->
       </joint>
     <joint name="hip_motorR_to_knee_motorR" type="fixed">
@@ -318,5 +318,5 @@
       <axis xyz="0.0 1.0 0.0"/>
       <dynamics damping="0.1" friction="0.0"/>
-      <!-- <limit effort="15.0" lower="${-PI}" upper="${PI}" velocity="30"/> -->
+      <limit effort="5.5" lower="${-PI}" upper="${PI}" velocity="30"/>
     </joint>
     <joint name="virtualhip_jointR" type="continuous">
@@ -326,5 +326,5 @@
       <axis xyz="0.0 1.0 0.0"/>
       <dynamics damping="0.1" friction="0.0"/>
-      <!-- <limit effort="15.0" lower="${-PI}" upper="${PI}" velocity="30"/> -->
+      <limit effort="5.5" lower="${-PI}" upper="${PI}" velocity="30"/>
     </joint>
     <joint name="wheel_jointR" type="continuous">
@@ -334,5 +334,5 @@
       <axis xyz="0.0 1.0 0.0"/>
       <dynamics damping="0.001" friction="0.0"/>
-      <limit effort="300.0" velocity="3000"/>
+      <limit effort="300.0" velocity="50"/>
     </joint>
     <gazebo reference="imu_link">

Commit message: zero velocity

File: otto_simulation/urdf/gazebo.xacro (robot description, xacro)
@@ -51,11 +51,13 @@
         <joint name="wheel_jointL">
             <command_interface name="effort">
-                <param name="min">-10000</param>
-                <param name="max">10000</param>
+                <param name="min">-10</param>
+                <param name="max">10</param>
               </command_interface>
               <state_interface name="position">
                 <param name="initial_value">0.0</param>
               </state_interface>
-              <state_interface name="velocity"/>
+              <state_interface name="velocity">
+                <param name="initial_value">0.0</param>
+              </state_interface>
               <state_interface name="effort"/>
         </joint>
@@ -97,11 +99,13 @@
         <joint name="wheel_jointR">
             <command_interface name="effort">
-                <param name="min">-10000</param>
-                <param name="max">10000</param>
+                <param name="min">-10</param>
+                <param name="max">10</param>
               </command_interface>
               <state_interface name="position">
                 <param name="initial_value">0.0</param>
               </state_interface>
-              <state_interface name="velocity"/>
+              <state_interface name="velocity">
+                <param name="initial_value">0.0</param>
+              </state_interface>
               <state_interface name="effort"/>
         </joint>
@@ -127,4 +131,7 @@
     <gazebo reference="leg_linkL">
         <material>Gazebo/Black</material>
+        <minDepth>0.0002</minDepth>
+        <kp  value="1000000.0"/>
+        <kd  value="100.0"/>
     </gazebo>
     <gazebo reference="wheel_linkL">
@@ -149,4 +156,7 @@
     <gazebo reference="leg_linkR">
         <material>Gazebo/Black</material>
+        <minDepth>0.0002</minDepth>
+        <kp  value="1000000.0"/>
+        <kd  value="100.0"/>
     </gazebo>
     <gazebo reference="wheel_linkR">

File: otto_simulation/urdf/otto-simulation.xacro (robot description, xacro)
@@ -37,5 +37,4 @@
       <child link="imu_link"/>
     </joint>
-    <!-- Camera -->
     <link name="imu_link">
       <inertial>
@@ -187,5 +186,5 @@
       <origin rpy="0.0 0.0 0.0" xyz="0.1414 0.02 -0.1414"/>
       <axis xyz="0.0 1.0 0.0"/>
-      <dynamics damping="0.001" friction="0.0"/>
+      <dynamics damping="0.01" friction="0.01"/>
       <limit effort="300.0" velocity="50"/>
     </joint>
@@ -333,5 +332,5 @@
       <origin rpy="0.0 0.0 0.0" xyz="0.1414 -0.02 -0.1414"/>
       <axis xyz="0.0 1.0 0.0"/>
-      <dynamics damping="0.001" friction="0.0"/>
+      <dynamics damping="0.01" friction="0.01"/>
       <limit effort="300.0" velocity="50"/>
     </joint>
