Commit message: forward kin

File: otto_simulation/urdf/gazebo.xacro (robot description, xacro)
@@ -26,6 +26,6 @@
                 <param name="max">10000</param>
               </command_interface> -->
-              <param name="pos_kp">100</param>
-              <param name="pos_ki">1</param>
+              <param name="pos_kp">300</param>
+              <param name="pos_ki">0</param>
               <param name="pos_kd">10</param>
               <param name="pos_max_integral_error">10000</param>
@@ -38,6 +38,6 @@
         </joint>
         <joint name="virtualhip_jointL">
-              <param name="pos_kp">100</param>
-              <param name="pos_ki">1</param>
+              <param name="pos_kp">300</param>
+              <param name="pos_ki">70</param>
               <param name="pos_kd">10</param>
               <param name="pos_max_integral_error">10000</param>
@@ -74,6 +74,6 @@
         </joint> -->
         <joint name="knee_jointR">
-              <param name="pos_kp">100</param>
-              <param name="pos_ki">1</param>
+              <param name="pos_kp">300</param>
+              <param name="pos_ki">0</param>
               <param name="pos_kd">10</param>
               <param name="pos_max_integral_error">10000</param>
@@ -86,6 +86,6 @@
         </joint>
         <joint name="virtualhip_jointR">
-              <param name="pos_kp">100</param>
-              <param name="pos_ki">1</param>
+              <param name="pos_kp">300</param>
+              <param name="pos_ki">70</param>
               <param name="pos_kd">10</param>
               <param name="pos_max_integral_error">10000</param>
@@ -136,6 +136,6 @@
     </gazebo>
     <gazebo reference="wheel_linkL">
-        <mu1>1.0</mu1>
-        <mu2>1.0</mu2>
+        <mu1>0.7</mu1>
+        <mu2>0.7</mu2>
         <minDepth>0.0002</minDepth>
         <kp  value="1000000.0"/>
@@ -161,6 +161,6 @@
     </gazebo>
     <gazebo reference="wheel_linkR">
-        <mu1>1.0</mu1>
-        <mu2>1.0</mu2>
+        <mu1>0.7</mu1>
+        <mu2>0.7</mu2>
         <minDepth>0.0002</minDepth>
         <kp  value="1000000.0"/>

File: otto_simulation/urdf/otto-simulation.xacro (robot description, xacro)
@@ -153,5 +153,5 @@
         <origin rpy="0.0 0.0 0.0" xyz="-0.03 0.06 0.0"/>
         <axis xyz="0.0 1.0 0.0"/>
-        <!-- <limit effort="50.0" lower="${-PI}" upper="${PI}" velocity="30"/> -->
+        <!-- <limit effort="4.0"="50.0" lower="${-PI}" upper="${PI}" velocity="30"/> -->
     </joint>
     <joint name="hip_motorL_to_knee_motorL" type="fixed">
@@ -171,5 +171,5 @@
       <axis xyz="0.0 1.0 0.0"/>
       <dynamics damping="0.1" friction="0.0"/>
-      <limit effort="5.5" lower="${-PI}" upper="${PI}" velocity="30"/>
+      <limit effort="4.0" lower="${-PI}" upper="${PI}" velocity="30"/>
     </joint>
     <joint name="virtualhip_jointL" type="continuous">
@@ -179,5 +179,5 @@
       <axis xyz="0.0 1.0 0.0"/>
       <dynamics damping="0.1" friction="0.0"/>
-      <limit effort="5.5" lower="${-PI}" upper="${PI}" velocity="30"/>
+      <limit effort="4.0" lower="${-PI}" upper="${PI}" velocity="30"/>
     </joint>
     <joint name="wheel_jointL" type="continuous">
@@ -317,5 +317,5 @@
       <axis xyz="0.0 1.0 0.0"/>
       <dynamics damping="0.1" friction="0.0"/>
-      <limit effort="5.5" lower="${-PI}" upper="${PI}" velocity="30"/>
+      <limit effort="4.0" lower="${-PI}" upper="${PI}" velocity="30"/>
     </joint>
     <joint name="virtualhip_jointR" type="continuous">
@@ -325,5 +325,5 @@
       <axis xyz="0.0 1.0 0.0"/>
       <dynamics damping="0.1" friction="0.0"/>
-      <limit effort="5.5" lower="${-PI}" upper="${PI}" velocity="30"/>
+      <limit effort="4.0" lower="${-PI}" upper="${PI}" velocity="30"/>
     </joint>
     <joint name="wheel_jointR" type="continuous">

Commit message: not fine tune

File: otto_simulation/urdf/gazebo.xacro (robot description, xacro)
@@ -26,7 +26,7 @@
                 <param name="max">10000</param>
               </command_interface> -->
-              <param name="pos_kp">300</param>
-              <param name="pos_ki">0</param>
-              <param name="pos_kd">10</param>
+              <param name="pos_kp">250</param>
+              <param name="pos_ki">20</param>
+              <param name="pos_kd">8</param>
               <param name="pos_max_integral_error">10000</param>
               <command_interface name="position_pid"/>
@@ -74,7 +74,7 @@
         </joint> -->
         <joint name="knee_jointR">
-              <param name="pos_kp">300</param>
-              <param name="pos_ki">0</param>
-              <param name="pos_kd">10</param>
+              <param name="pos_kp">250</param>
+              <param name="pos_ki">20</param>
+              <param name="pos_kd">8</param>
               <param name="pos_max_integral_error">10000</param>
               <command_interface name="position_pid"/>
@@ -136,6 +136,6 @@
     </gazebo>
     <gazebo reference="wheel_linkL">
-        <mu1>0.7</mu1>
-        <mu2>0.7</mu2>
+        <mu1>1.2</mu1>
+        <mu2>1.2</mu2>
         <minDepth>0.0002</minDepth>
         <kp  value="1000000.0"/>
@@ -161,6 +161,6 @@
     </gazebo>
     <gazebo reference="wheel_linkR">
-        <mu1>0.7</mu1>
-        <mu2>0.7</mu2>
+        <mu1>1.2</mu1>
+        <mu2>1.2</mu2>
         <minDepth>0.0002</minDepth>
         <kp  value="1000000.0"/>

File: otto_simulation/urdf/otto-simulation.xacro (robot description, xacro)
@@ -4,10 +4,10 @@
     <xacro:property name="PI" value="3.14159265359"/>
     <xacro:include filename="gazebo.xacro"/>
-    <link name="world"></link>
+    <!-- <link name="world"></link>
     <joint name="base_joint" type="fixed">
       <origin xyz="0.0 0.0 0.5" rpy="0.0 0.0 0.0"/>
       <parent link="world"/>
       <child link="base_link"/>
-    </joint>
+    </joint> -->
     <!-- Base Link -->
     <link name="base_link">
@@ -153,5 +153,5 @@
         <origin rpy="0.0 0.0 0.0" xyz="-0.03 0.06 0.0"/>
         <axis xyz="0.0 1.0 0.0"/>
-        <!-- <limit effort="4.0"="50.0" lower="${-PI}" upper="${PI}" velocity="30"/> -->
+        <!-- <limit effort="8.0"="50.0" lower="${-PI}" upper="${PI}" velocity="30"/> -->
     </joint>
     <joint name="hip_motorL_to_knee_motorL" type="fixed">
@@ -170,6 +170,6 @@
       <origin rpy="0.0 0.0 0.0" xyz="0.0 0.055 0.0"/>
       <axis xyz="0.0 1.0 0.0"/>
-      <dynamics damping="0.1" friction="0.0"/>
-      <limit effort="4.0" lower="${-PI}" upper="${PI}" velocity="30"/>
+      <dynamics damping="0.22" friction="0.0"/>
+      <limit effort="8.0" lower="${-PI}" upper="${PI}" velocity="30"/>
     </joint>
     <joint name="virtualhip_jointL" type="continuous">
@@ -178,6 +178,6 @@
       <origin rpy="0.0 0.0 0.0" xyz="-0.1414 -0.05 -0.1414"/>
       <axis xyz="0.0 1.0 0.0"/>
-      <dynamics damping="0.1" friction="0.0"/>
-      <limit effort="4.0" lower="${-PI}" upper="${PI}" velocity="30"/>
+      <dynamics damping="0.22" friction="0.0"/>
+      <limit effort="8.0" lower="${-PI}" upper="${PI}" velocity="30"/>
     </joint>
     <joint name="wheel_jointL" type="continuous">
@@ -316,6 +316,6 @@
       <origin rpy="0.0 0.0 0.0" xyz="0.0 -0.055 0.0"/>
       <axis xyz="0.0 1.0 0.0"/>
-      <dynamics damping="0.1" friction="0.0"/>
-      <limit effort="4.0" lower="${-PI}" upper="${PI}" velocity="30"/>
+      <dynamics damping="0.22" friction="0.0"/>
+      <limit effort="8.0" lower="${-PI}" upper="${PI}" velocity="30"/>
     </joint>
     <joint name="virtualhip_jointR" type="continuous">
@@ -324,6 +324,6 @@
       <origin rpy="0.0 0.0 0.0" xyz="-0.1414 0.05 -0.1414"/>
       <axis xyz="0.0 1.0 0.0"/>
-      <dynamics damping="0.1" friction="0.0"/>
-      <limit effort="4.0" lower="${-PI}" upper="${PI}" velocity="30"/>
+      <dynamics damping="0.22" friction="0.0"/>
+      <limit effort="8.0" lower="${-PI}" upper="${PI}" velocity="30"/>
     </joint>
     <joint name="wheel_jointR" type="continuous">

Commit message: jump I

File: otto_simulation/urdf/gazebo.xacro (robot description, xacro)
@@ -27,5 +27,5 @@
               </command_interface> -->
               <param name="pos_kp">220</param>
-              <param name="pos_ki">0</param>
+              <param name="pos_ki">20</param>
               <param name="pos_kd">8</param>
               <param name="pos_max_integral_error">10000</param>
@@ -39,5 +39,5 @@
         <joint name="virtualhip_jointL">
               <param name="pos_kp">300</param>
-              <param name="pos_ki">0</param>
+              <param name="pos_ki">70</param>
               <param name="pos_kd">10</param>
               <param name="pos_max_integral_error">10000</param>
@@ -51,6 +51,6 @@
         <joint name="wheel_jointL">
             <command_interface name="effort">
-                <param name="min">-5</param>
-                <param name="max">5</param>
+                <param name="min">-10</param>
+                <param name="max">10</param>
               </command_interface>
               <state_interface name="position">
@@ -75,5 +75,5 @@
         <joint name="knee_jointR">
               <param name="pos_kp">220</param>
-              <param name="pos_ki">0</param>
+              <param name="pos_ki">20</param>
               <param name="pos_kd">8</param>
               <param name="pos_max_integral_error">10000</param>
@@ -87,5 +87,5 @@
         <joint name="virtualhip_jointR">
               <param name="pos_kp">300</param>
-              <param name="pos_ki">0</param>
+              <param name="pos_ki">70</param>
               <param name="pos_kd">10</param>
               <param name="pos_max_integral_error">10000</param>
@@ -99,6 +99,6 @@
         <joint name="wheel_jointR">
             <command_interface name="effort">
-                <param name="min">-5</param>
-                <param name="max">5</param>
+                <param name="min">-10</param>
+                <param name="max">10</param>
               </command_interface>
               <state_interface name="position">
@@ -124,11 +124,11 @@
     </gazebo>
     <gazebo reference="hip_linkL">
-        <material>Gazebo/Black</material>
+        <material>Gazebo/FlatBlack</material>
     </gazebo>
     <gazebo reference="knee_linkL">
-        <material>Gazebo/Black</material>
+        <material>Gazebo/FlatBlack</material>
     </gazebo>
     <gazebo reference="leg_linkL">
-        <material>Gazebo/Black</material>
+        <material>Gazebo/FlatBlack</material>
         <minDepth>0.0002</minDepth>
         <kp  value="1000000.0"/>
@@ -136,8 +136,8 @@
     </gazebo>
     <gazebo reference="wheel_linkL">
-        <mu1>10.0</mu1>
-        <mu2>10.0</mu2>
+        <mu1>1.5</mu1>
+        <mu2>1.5</mu2>
         <minDepth>0.0002</minDepth>
-        <kp  value="1000000.0"/>
+        <kp  value="10000.0"/>
         <kd  value="1000.0"/>
     </gazebo>
@@ -149,21 +149,21 @@
     </gazebo>
     <gazebo reference="hip_linkR">
-        <material>Gazebo/Black</material>
+        <material>Gazebo/FlatBlack</material>
     </gazebo>
     <gazebo reference="knee_linkR">
-        <material>Gazebo/Black</material>
+        <material>Gazebo/FlatBlack</material>
     </gazebo>
     <gazebo reference="leg_linkR">
-        <material>Gazebo/Black</material>
-        <minDepth>0.0002</minDepth>
-        <kp  value="1000000.0"/>
-        <kd  value="1000.0"/>
-    </gazebo>
-    <gazebo reference="wheel_linkR">
-        <mu1>10.0</mu1>
-        <mu2>10.0</mu2>
+        <material>Gazebo/FlatBlack</material>
         <minDepth>0.0002</minDepth>
         <kp  value="1000000.0"/>
         <kd  value="100.0"/>
     </gazebo>
+    <gazebo reference="wheel_linkR">
+        <mu1>1.5</mu1>
+        <mu2>1.5</mu2>
+        <minDepth>0.0002</minDepth>
+        <kp  value="10000.0"/>
+        <kd  value="1000.0"/>
+    </gazebo>
 </robot>

File: otto_simulation/urdf/gazebotest.xacro (robot description, xacro)
@@ -12,6 +12,6 @@
         <joint name="wheel_jointL">
             <command_interface name="effort">
-                <param name="min">-5</param>
-                <param name="max">5</param>
+                <param name="min">-10000</param>
+                <param name="max">10000</param>
               </command_interface>
               <state_interface name="position">
@@ -23,6 +23,6 @@
         <joint name="wheel_jointR">
             <command_interface name="effort">
-                <param name="min">-5</param>
-                <param name="max">5</param>
+                <param name="min">-10000</param>
+                <param name="max">10000</param>
               </command_interface>
               <state_interface name="position">
@@ -55,8 +55,8 @@
     </gazebo>
     <gazebo reference="wheel_linkL">
-        <mu1>2.0</mu1>
-        <mu2>2.0</mu2>
+        <mu1>1.0</mu1>
+        <mu2>1.0</mu2>
         <minDepth>0.0002</minDepth>
-        <kp  value="1000000.0"/>
+        <kp  value="100000.0"/>
         <kd  value="100.0"/>
     </gazebo>
@@ -77,8 +77,8 @@
     </gazebo>
     <gazebo reference="wheel_linkR">
-        <mu1>2.0</mu1>
-        <mu2>2.0</mu2>
+        <mu1>1.0</mu1>
+        <mu2>1.0</mu2>
         <minDepth>0.0002</minDepth>
-        <kp  value="1000000.0"/>
+        <kp  value="100000.0"/>
         <kd  value="100.0"/>
     </gazebo>

File: otto_simulation/urdf/otto-simulation.xacro (robot description, xacro)
@@ -13,6 +13,8 @@
     <link name="base_link">
         <inertial>
-          <origin xyz="-0.02195199 0.0 0.0" rpy="0 0 0"/>
-          <mass value="3.00"/>
+          <!-- <origin xyz="-0.02195199 0.0 0.0" rpy="0 0 0"/>
+          <mass value="3.0"/> -->
+          <origin xyz="-0.0136 0.0 0.0" rpy="0 0 0"/>
+          <mass value="1.5"/>
           <inertia ixx="14584893e-9" ixy="0.0" ixz="0.0"
                    iyx="0.0" iyy="16663530e-9" iyz="0.0"
@@ -33,5 +35,4 @@
     </link>
     <joint name="imu_joint" type="fixed">
-      <axis xyz="0 1 0" />
       <parent link="base_link"/>
       <child link="imu_link"/>
@@ -40,5 +41,5 @@
       <inertial>
         <mass value="1e-5" />
-        <origin xyz="0 0 0" rpy="0 0 0"/>
+        <origin xyz="-0.03 0 0" rpy="0 0 0"/>
         <inertia ixx="1e-6" ixy="0" ixz="0" iyy="1e-6" iyz="0" izz="1e-6" />
       </inertial>
@@ -142,7 +143,7 @@
       </visual>
       <collision>
-        <origin rpy="${PI/2} 0.0 0.0" xyz="0.0 0.02 0.0"/>
+        <origin rpy="${PI/2} 0.0 0.0" xyz="0.0 0.04 0.0"/>
         <geometry>
-            <cylinder radius="0.086" length="0.04416"/>
+            <cylinder radius="0.086" length="0.07416"/>
         </geometry>
       </collision>
@@ -288,7 +289,7 @@
       </visual>
       <collision>
-        <origin rpy="${PI/2} 0.0 0.0" xyz="0.0 -0.02 0.0"/>
+        <origin rpy="${PI/2} 0.0 0.0" xyz="0.0 -0.04 0.0"/>
         <geometry>
-            <cylinder radius="0.086" length="0.04416"/>
+            <cylinder radius="0.086" length="0.07416"/>
         </geometry>
       </collision>
@@ -354,3 +355,90 @@
       </sensor>
     </gazebo>
+    <!-- LiDAR Sensor -->
+    <link name="lidar_link"/>
+    <joint name="lidar_joint" type="fixed">
+        <parent link="base_link"/>
+        <child link="lidar_link"/>
+        <origin xyz="0 0 -0.15" rpy="0 0 0"/>
+    </joint>
+    <gazebo reference="lidar_link">
+        <sensor type="ray" name="laser_sensor">
+          <pose>0 0 0 0 0 0</pose>
+          <visualize>false</visualize>
+          <update_rate>8</update_rate>
+          <ray>
+            <scan>
+              <horizontal>
+                <samples>720</samples>
+                <resolution>1</resolution>
+                <min_angle>-3.14</min_angle>
+                <max_angle>3.14</max_angle>
+              </horizontal>
+            </scan>
+            <range>
+              <min>1.0</min>
+              <max>8.0</max>
+              <resolution>0.01</resolution>
+            </range>
+            <noise>
+              <type>gaussian</type>
+              <mean>0.0</mean>
+              <stddev>0.01</stddev>
+            </noise>
+          </ray>
+          <plugin name="gazebo_ros_laser_sensor" filename="libgazebo_ros_ray_sensor.so">
+          <ros>
+            <remapping>~/out:=scan</remapping>
+          </ros>
+            <topicName>/scan</topicName>
+            <frameName>laser_link</frameName>
+          </plugin>
+        </sensor>
+    </gazebo>
+    <!-- Depth Camera -->
+    <link name="depth_link"/>
+    <joint name="depth_camera_joint" type="fixed">
+        <parent link="base_link"/>
+        <child link="depth_link"/>
+        <origin xyz="0.05 0 0.1" rpy="0 0 0"/>
+    </joint>
+    <link name="camera_depth_optical_frame"/>
+    <joint name="camera_depth_optical_joint" type="fixed">
+      <origin xyz="0 0 0" rpy="-1.57 0 -1.57" />
+      <parent link="depth_link" />
+      <child link="camera_depth_optical_frame" />
+    </joint>
+    <gazebo reference="depth_link">
+          <sensor name="sensor_camera" type="depth">
+            <pose>0.0 0.0 0.0 0.0 0.0 0.0</pose>
+            <always_on>1</always_on>
+            <update_rate>10</update_rate>
+            <visualize>1</visualize>
+            <camera name="limo_camera">
+              <image>
+                <format>R8G8B8</format>
+                <width>400</width>
+                <height>400</height>
+              </image>
+              <clip>
+                <near>0.01</near>
+                <far>10.0</far>
+              </clip>
+            </camera>
+            <plugin name="gazebo_ros_depth_camera_sensor" filename="libgazebo_ros_camera.so">
+              <ros>
+                <namespace>/limo</namespace>
+                <argument>limo_camera/image_raw:=limo_camera/image</argument>
+                <argument>limo_camera/image_depth:=limo_camera/depth/camera_image_depth</argument>
+                <argument>limo_camera/camera_info:=limo_camera/camera_info_raw</argument>
+                <argument>limo_camera/camera_info_depth:=limo_camera/camera_info_depth</argument>
+                <argument>limo_camera/points:=limo_camera/camera_points</argument>
+              </ros>
+              <camera_name>depth_link</camera_name>
+              <frame_name>camera_depth_optical_frame</frame_name>
+              <hack_baseline>0.07</hack_baseline>
+              <min_depth>0.001</min_depth>
+            </plugin>
+        </sensor>
+    </gazebo>
 </robot>

Commit message: add ramp

File: otto_simulation/urdf/gazebo.xacro (robot description, xacro)
@@ -135,10 +135,13 @@
         <kd  value="100.0"/>
     </gazebo>
-    <gazebo reference="wheel_linkL">
-        <mu1>1.5</mu1>
-        <mu2>1.5</mu2>
+    <gazebo reference="wheel_linkR">
+        <mu1>2.0</mu1>
+        <mu2>2.0</mu2>
         <minDepth>0.0002</minDepth>
-        <kp  value="10000.0"/>
-        <kd  value="1000.0"/>
+        <kp>100000.0</kp>
+        <kd>10000.0</kd>
+        <material>default</material>
+        <maxVel>0.0</maxVel>
+        <restitution_coefficient>0.0</restitution_coefficient>
     </gazebo>
     <gazebo reference="hip_motorR">
@@ -161,9 +164,12 @@
     </gazebo>
     <gazebo reference="wheel_linkR">
-        <mu1>1.5</mu1>
-        <mu2>1.5</mu2>
+        <mu1>2.0</mu1>
+        <mu2>2.0</mu2>
         <minDepth>0.0002</minDepth>
-        <kp  value="10000.0"/>
-        <kd  value="1000.0"/>
+        <kp>100000.0</kp>
+        <kd>10000.0</kd>
+        <material>default</material>
+        <maxVel>0.0</maxVel>
+        <restitution_coefficient>0.0</restitution_coefficient>
     </gazebo>
 </robot>
