Commit message: seem stable

File: otto_simulation/urdf/gazebo.xacro (robot description, xacro)
@@ -135,12 +135,10 @@
         <kd  value="100.0"/>
     </gazebo>
-    <gazebo reference="wheel_linkR">
-        <mu1>2.0</mu1>
-        <mu2>2.0</mu2>
+    <gazebo reference="wheel_linkL">
+        <mu1>1.5</mu1>
+        <mu2>1.5</mu2>
         <minDepth>0.0002</minDepth>
-        <kp>100000.0</kp>
-        <kd>10000.0</kd>
-        <material>default</material>
-        <maxVel>0.0</maxVel>
+        <kp  value="1000000.0"/>
+        <kd  value="100.0"/>
         <restitution_coefficient>0.0</restitution_coefficient>
     </gazebo>
@@ -163,13 +161,11 @@
         <kd  value="100.0"/>
     </gazebo>
-    <gazebo reference="wheel_linkR">
-        <mu1>2.0</mu1>
-        <mu2>2.0</mu2>
-        <minDepth>0.0002</minDepth>
-        <kp>100000.0</kp>
-        <kd>10000.0</kd>
-        <material>default</material>
-        <maxVel>0.0</maxVel>
-        <restitution_coefficient>0.0</restitution_coefficient>
-    </gazebo>
+<gazebo reference="wheel_linkR">
+    <mu1>1.5</mu1>
+    <mu2>1.5</mu2>
+    <minDepth>0.0002</minDepth>
+    <kp  value="1000000.0"/>
+    <kd  value="100.0"/>
+    <restitution_coefficient>0.0</restitution_coefficient>
+</gazebo>
 </robot>

File: otto_simulation/urdf/otto-simulation.xacro (robot description, xacro)
@@ -143,7 +143,7 @@
       </visual>
       <collision>
-        <origin rpy="${PI/2} 0.0 0.0" xyz="0.0 0.04 0.0"/>
+        <origin rpy="${PI/2} 0.0 0.0" xyz="0.0 0.0 0.0"/>
         <geometry>
-            <cylinder radius="0.086" length="0.07416"/>
+            <cylinder radius="0.086" length="0.0001"/>
         </geometry>
       </collision>
@@ -154,5 +154,5 @@
         <origin rpy="0.0 0.0 0.0" xyz="-0.03 0.06 0.0"/>
         <axis xyz="0.0 1.0 0.0"/>
-        <!-- <limit effort="8.0"="50.0" lower="${-PI}" upper="${PI}" velocity="30"/> -->
+        <!-- <limit effort="10.0"="50.0" lower="${-PI}" upper="${PI}" velocity="60"/> -->
     </joint>
     <joint name="hip_motorL_to_knee_motorL" type="fixed">
@@ -172,5 +172,5 @@
       <axis xyz="0.0 1.0 0.0"/>
       <dynamics damping="0.22" friction="0.0"/>
-      <limit effort="8.0" lower="${-PI}" upper="${PI}" velocity="30"/>
+      <limit effort="10.0" velocity="60"/>
     </joint>
     <joint name="virtualhip_jointL" type="continuous">
@@ -180,5 +180,5 @@
       <axis xyz="0.0 1.0 0.0"/>
       <dynamics damping="0.22" friction="0.0"/>
-      <limit effort="8.0" lower="${-PI}" upper="${PI}" velocity="30"/>
+      <limit effort="10.0" velocity="60"/>
     </joint>
     <joint name="wheel_jointL" type="continuous">
@@ -289,7 +289,7 @@
       </visual>
       <collision>
-        <origin rpy="${PI/2} 0.0 0.0" xyz="0.0 -0.04 0.0"/>
+        <origin rpy="${PI/2} 0.0 0.0" xyz="0.0 -0.0 0.0"/>
         <geometry>
-            <cylinder radius="0.086" length="0.07416"/>
+            <cylinder radius="0.086" length="0.0001"/>
         </geometry>
       </collision>
@@ -300,5 +300,5 @@
         <origin rpy="0.0 0.0 0.0" xyz="-0.03 -0.06 0.0"/>
         <axis xyz="0.0 1.0 0.0"/>
-        <!-- <limit effort="5.0" lower="${-PI}" upper="${PI}" velocity="30"/> -->
+        <!-- <limit effort="5.0" lower="${-PI}" upper="${PI}" velocity="60"/> -->
       </joint>
     <joint name="hip_motorR_to_knee_motorR" type="fixed">
@@ -318,5 +318,5 @@
       <axis xyz="0.0 1.0 0.0"/>
       <dynamics damping="0.22" friction="0.0"/>
-      <limit effort="8.0" lower="${-PI}" upper="${PI}" velocity="30"/>
+      <limit effort="10.0" velocity="60"/>
     </joint>
     <joint name="virtualhip_jointR" type="continuous">
@@ -326,5 +326,5 @@
       <axis xyz="0.0 1.0 0.0"/>
       <dynamics damping="0.22" friction="0.0"/>
-      <limit effort="8.0" lower="${-PI}" upper="${PI}" velocity="30"/>
+      <limit effort="10.0" velocity="60"/>
     </joint>
     <joint name="wheel_jointR" type="continuous">
@@ -340,5 +340,5 @@
       <sensor name="imu_sensor" type="imu">
         <always_on>true</always_on>
-        <update_rate>500.0</update_rate>
+        <update_rate>3000.0</update_rate>
         <visualize>true</visualize>
         <plugin filename="libgazebo_ros_imu_sensor.so" name="imu_plugin">
@@ -356,5 +356,5 @@
     </gazebo>
     <!-- LiDAR Sensor -->
-    <link name="lidar_link"/>
+    <!-- <link name="lidar_link"/>
     <joint name="lidar_joint" type="fixed">
         <parent link="base_link"/>
@@ -395,7 +395,7 @@
           </plugin>
         </sensor>
-    </gazebo>
+    </gazebo> -->
     <!-- Depth Camera -->
-    <link name="depth_link"/>
+    <!-- <link name="depth_link"/>
     <joint name="depth_camera_joint" type="fixed">
         <parent link="base_link"/>
@@ -441,4 +441,4 @@
             </plugin>
         </sensor>
-    </gazebo>
+    </gazebo> -->
 </robot>

Commit message: hyper damp

File: otto_simulation/urdf/gazebo.xacro (robot description, xacro)
@@ -22,29 +22,27 @@
         </joint> -->
         <joint name="knee_jointL">
-            <!-- <command_interface name="effort">
-                <param name="min">-10000</param>
-                <param name="max">10000</param>
-              </command_interface> -->
-              <param name="pos_kp">220</param>
-              <param name="pos_ki">20</param>
-              <param name="pos_kd">8</param>
-              <param name="pos_max_integral_error">10000</param>
-              <command_interface name="position_pid"/>
+            <command_interface name="effort">
+                <param name="min">-10</param>
+                <param name="max">10</param>
+              </command_interface>
               <state_interface name="position">
                 <param name="initial_value">0.0</param>
               </state_interface>
-              <state_interface name="velocity"/>
+              <state_interface name="velocity">
+                <param name="initial_value">0.0</param>
+              </state_interface>
               <state_interface name="effort"/>
         </joint>
         <joint name="virtualhip_jointL">
-              <param name="pos_kp">300</param>
-              <param name="pos_ki">70</param>
-              <param name="pos_kd">10</param>
-              <param name="pos_max_integral_error">10000</param>
-              <command_interface name="position_pid"/>
+            <command_interface name="effort">
+                <param name="min">-10</param>
+                <param name="max">10</param>
+              </command_interface>
               <state_interface name="position">
                 <param name="initial_value">0.0</param>
               </state_interface>
-              <state_interface name="velocity"/>
+              <state_interface name="velocity">
+                <param name="initial_value">0.0</param>
+              </state_interface>
               <state_interface name="effort"/>
         </joint>
@@ -62,37 +60,28 @@
               <state_interface name="effort"/>
         </joint>
-        <!-- <joint name="hip_jointR">
+        <joint name="knee_jointR">
             <command_interface name="effort">
-                <param name="min">-10000</param>
-                <param name="max">10000</param>
+                <param name="min">-10</param>
+                <param name="max">10</param>
               </command_interface>
               <state_interface name="position">
                 <param name="initial_value">0.0</param>
               </state_interface>
-              <state_interface name="velocity"/>
+              <state_interface name="velocity">
+                <param name="initial_value">0.0</param>
+              </state_interface>
               <state_interface name="effort"/>
-        </joint> -->
-        <joint name="knee_jointR">
-              <param name="pos_kp">220</param>
-              <param name="pos_ki">20</param>
-              <param name="pos_kd">8</param>
-              <param name="pos_max_integral_error">10000</param>
-              <command_interface name="position_pid"/>
+        </joint>
+        <joint name="virtualhip_jointR">
+            <command_interface name="effort">
+                <param name="min">-10</param>
+                <param name="max">10</param>
+              </command_interface>
               <state_interface name="position">
                 <param name="initial_value">0.0</param>
               </state_interface>
-              <state_interface name="velocity"/>
-              <state_interface name="effort"/>
-        </joint>
-        <joint name="virtualhip_jointR">
-              <param name="pos_kp">300</param>
-              <param name="pos_ki">70</param>
-              <param name="pos_kd">10</param>
-              <param name="pos_max_integral_error">10000</param>
-              <command_interface name="position_pid"/>
-              <state_interface name="position">
+              <state_interface name="velocity">
                 <param name="initial_value">0.0</param>
               </state_interface>
-              <state_interface name="velocity"/>
               <state_interface name="effort"/>
         </joint>

File: otto_simulation/urdf/otto-simulation.xacro (robot description, xacro)
@@ -172,5 +172,5 @@
       <origin rpy="0.0 0.0 0.0" xyz="0.0 0.055 0.0"/>
       <axis xyz="0.0 1.0 0.0"/>
-      <dynamics damping="0.22" friction="0.0"/>
+      <dynamics damping="0.85" friction="0.05"/>
       <limit effort="10.0" velocity="60"/>
     </joint>
@@ -180,5 +180,5 @@
       <origin rpy="0.0 0.0 0.0" xyz="-0.1414 -0.05 -0.1414"/>
       <axis xyz="0.0 1.0 0.0"/>
-      <dynamics damping="0.22" friction="0.0"/>
+      <dynamics damping="0.85" friction="0.05"/>
       <limit effort="10.0" velocity="60"/>
     </joint>
@@ -318,5 +318,5 @@
       <origin rpy="0.0 0.0 0.0" xyz="0.0 -0.055 0.0"/>
       <axis xyz="0.0 1.0 0.0"/>
-      <dynamics damping="0.22" friction="0.0"/>
+      <dynamics damping="0.85" friction="0.05"/>
       <limit effort="10.0" velocity="60"/>
     </joint>
@@ -326,5 +326,5 @@
       <origin rpy="0.0 0.0 0.0" xyz="-0.1414 0.05 -0.1414"/>
       <axis xyz="0.0 1.0 0.0"/>
-      <dynamics damping="0.22" friction="0.0"/>
+      <dynamics damping="0.85" friction="0.05"/>
       <limit effort="10.0" velocity="60"/>
     </joint>
