Commit message: delete dummy

File: otto_simulation/urdf/otto-simulation.xacro (robot description, xacro)
@@ -6,5 +6,5 @@
     <link name="world"></link>
     <joint name="base_joint" type="fixed">
-      <origin xyz="0 0 0.3" rpy="0 0 0"/>
+      <origin xyz="0.0 0.0 0.0" rpy="0.0 0.0 0.0"/>
       <parent link="world"/>
       <child link="base_link"/>

Commit message: read feedback

File: otto_simulation/urdf/otto-simulation.xacro (robot description, xacro)
@@ -136,5 +136,5 @@
         <axis xyz="0.0 1.0 0.0"/>
       <dynamics damping="0.1" friction="0.05"/>
-      <limit effort="1000.0" lower="${PI}" upper="${-PI}" velocity="30"/>
+      <limit effort="100.0" lower="${PI}" upper="${-PI}" velocity="30"/>
     </joint>
     <joint name="hip_motorL_to_knee_motorL" type="fixed">
@@ -154,5 +154,5 @@
       <axis xyz="0.0 1.0 0.0"/>
       <dynamics damping="0.1" friction="0.05"/>
-      <limit effort="1000.0" lower="${PI}" upper="${-PI}" velocity="30"/>
+      <limit effort="100.0" lower="${PI}" upper="${-PI}" velocity="30"/>
     </joint>
     <joint name="virtualhip_jointL" type="continuous">
@@ -162,5 +162,5 @@
       <axis xyz="0.0 1.0 0.0"/>
       <dynamics damping="0.1" friction="0.05"/>
-      <limit effort="1000.0" lower="${PI}" upper="${-PI}" velocity="30"/>
+      <limit effort="100.0" lower="${PI}" upper="${-PI}" velocity="30"/>
     </joint>
     <joint name="wheel_jointL" type="continuous">
@@ -170,5 +170,5 @@
       <axis xyz="0.0 1.0 0.0"/>
       <dynamics damping="0.1" friction="0.05"/>
-      <limit effort="1000.0" velocity="30"/>
+      <limit effort="100.0" velocity="30"/>
     </joint>
     <!-- Right Side -->
@@ -277,5 +277,5 @@
         <axis xyz="0.0 1.0 0.0"/>
         <dynamics damping="0.1" friction="0.05"/>
-        <limit effort="1000.0" lower="${PI}" upper="${-PI}" velocity="30"/>
+        <limit effort="100.0" lower="${PI}" upper="${-PI}" velocity="30"/>
     </joint>
     <joint name="hip_motorR_to_knee_motorR" type="fixed">
@@ -295,5 +295,5 @@
       <axis xyz="0.0 1.0 0.0"/>
       <dynamics damping="0.1" friction="0.05"/>
-      <limit effort="1000.0" lower="${PI}" upper="${-PI}" velocity="30"/>
+      <limit effort="100.0" lower="${PI}" upper="${-PI}" velocity="30"/>
     </joint>
     <joint name="virtualhip_jointR" type="continuous">
@@ -303,5 +303,5 @@
       <axis xyz="0.0 1.0 0.0"/>
       <dynamics damping="0.1" friction="0.05"/>
-      <limit effort="1000.0" lower="${PI}" upper="${-PI}" velocity="30"/>
+      <limit effort="100.0" lower="${PI}" upper="${-PI}" velocity="30"/>
     </joint>
     <joint name="wheel_jointR" type="continuous">
@@ -311,5 +311,5 @@
       <axis xyz="0.0 1.0 0.0"/>
       <dynamics damping="0.1" friction="0.05"/>
-      <limit effort="1000.0" velocity="30"/>
+      <limit effort="100.0" velocity="30"/>
     </joint>
 </robot>

Commit message: add exit

File: otto_simulation/urdf/otto-simulation.xacro (robot description, xacro)
@@ -6,5 +6,5 @@
     <link name="world"></link>
     <joint name="base_joint" type="fixed">
-      <origin xyz="0.0 0.0 0.0" rpy="0.0 0.0 0.0"/>
+      <origin xyz="0.0 0.0 0.5" rpy="0.0 0.0 0.0"/>
       <parent link="world"/>
       <child link="base_link"/>

Commit message: add imu

File: otto_simulation/urdf/otto-simulation.xacro (robot description, xacro)
@@ -32,4 +32,17 @@
         </collision>
     </link>
+    <joint name="imu_joint" type="fixed">
+      <axis xyz="0 1 0" />
+      <parent link="base_link"/>
+      <child link="imu_link"/>
+    </joint>
+    <!-- Camera -->
+    <link name="imu_link">
+      <inertial>
+        <mass value="1e-5" />
+        <origin xyz="0 0 0" rpy="0 0 0"/>
+        <inertia ixx="1e-6" ixy="0" ixz="0" iyy="1e-6" iyz="0" izz="1e-6" />
+      </inertial>
+    </link>
     <!-- Hip Motor Left -->
     <link name="hip_motorL">
@@ -142,5 +155,5 @@
         <axis xyz="0.0 1.0 0.0"/>
       <dynamics damping="0.2" friction="0.05"/>
-      <limit effort="100.0" lower="${PI}" upper="${-PI}" velocity="30"/>
+      <limit effort="15.0" lower="${-PI}" upper="${PI}" velocity="30"/>
     </joint>
     <joint name="hip_motorL_to_knee_motorL" type="fixed">
@@ -160,5 +173,5 @@
       <axis xyz="0.0 1.0 0.0"/>
       <dynamics damping="0.1" friction="0.02"/>
-      <limit effort="100.0" lower="${PI}" upper="${-PI}" velocity="30"/>
+      <limit effort="15.0" lower="${-PI}" upper="${PI}" velocity="30"/>
     </joint>
     <joint name="virtualhip_jointL" type="revolute">
@@ -168,5 +181,5 @@
       <axis xyz="0.0 1.0 0.0"/>
       <dynamics damping="0.1" friction="0.05"/>
-      <limit effort="100.0" lower="${PI}" upper="${-PI}" velocity="30"/>
+      <limit effort="15.0" lower="${-PI}" upper="${PI}" velocity="30"/>
     </joint>
     <joint name="wheel_jointL" type="continuous">
@@ -289,6 +302,6 @@
         <axis xyz="0.0 1.0 0.0"/>
         <dynamics damping="0.2" friction="0.05"/>
-        <limit effort="100.0" lower="${PI}" upper="${-PI}" velocity="30"/>
-    </joint>
+        <limit effort="15.0" lower="${-PI}" upper="${PI}" velocity="30"/>
+      </joint>
     <joint name="hip_motorR_to_knee_motorR" type="fixed">
       <parent link="hip_motorR"/>
@@ -307,5 +320,5 @@
       <axis xyz="0.0 1.0 0.0"/>
       <dynamics damping="0.1" friction="0.02"/>
-      <limit effort="100.0" lower="${PI}" upper="${-PI}" velocity="30"/>
+      <limit effort="15.0" lower="${-PI}" upper="${PI}" velocity="30"/>
     </joint>
     <joint name="virtualhip_jointR" type="revolute">
@@ -315,5 +328,5 @@
       <axis xyz="0.0 1.0 0.0"/>
       <dynamics damping="0.1" friction="0.05"/>
-      <limit effort="100.0" lower="${PI}" upper="${-PI}" velocity="30"/>
+      <limit effort="15.0" lower="${-PI}" upper="${PI}" velocity="30"/>
     </joint>
     <joint name="wheel_jointR" type="continuous">
@@ -325,3 +338,22 @@
       <limit effort="100.0" velocity="30"/>
     </joint>
+    <gazebo reference="imu_link">
+      <gravity>true</gravity>
+      <sensor name="imu_sensor" type="imu">
+        <always_on>true</always_on>
+        <update_rate>1000</update_rate>
+        <visualize>true</visualize>
+        <plugin filename="libgazebo_ros_imu_sensor.so" name="imu_plugin">
+          <topicName>otto_imu</topicName>
+          <bodyName>imu_link</bodyName>
+          <updateRateHZ>1000.0</updateRateHZ>
+          <gaussianNoise>0.0</gaussianNoise>
+          <xyzOffset>0 0 0</xyzOffset>
+          <rpyOffset>0 0 0</rpyOffset>
+          <frameName>imu_link</frameName>
+          <initialOrientationAsReference>false</initialOrientationAsReference>
+        </plugin>
+        <pose>0 0 0 0 0 0</pose>
+      </sensor>
+    </gazebo>
 </robot>

Commit message: jacobian

File: otto_simulation/urdf/otto-simulation.xacro (robot description, xacro)
@@ -4,10 +4,10 @@
     <xacro:property name="PI" value="3.14159265359"/>
     <xacro:include filename="gazebo.xacro"/>
-    <!-- <link name="world"></link>
+    <link name="world"></link>
     <joint name="base_joint" type="fixed">
       <origin xyz="0.0 0.0 0.5" rpy="0.0 0.0 0.0"/>
       <parent link="world"/>
       <child link="base_link"/>
-    </joint> -->
+    </joint>
     <!-- Base Link -->
     <link name="base_link">

Commit message: up down slope

File: otto_simulation/urdf/otto-simulation.xacro (robot description, xacro)
@@ -4,5 +4,6 @@
     <xacro:property name="PI" value="3.14159265359"/>
     <xacro:include filename="gazebo.xacro"/>
-    <!-- <link name="world"></link>
+    <!-- <link name="world"></link> -->
+<!--
     <joint name="base_joint" type="fixed">
       <origin xyz="0.0 0.0 0.5" rpy="0.0 0.0 0.0"/>
@@ -340,10 +341,10 @@
       <sensor name="imu_sensor" type="imu">
         <always_on>true</always_on>
-        <update_rate>3000.0</update_rate>
+        <update_rate>2000.0</update_rate>
         <visualize>true</visualize>
         <plugin filename="libgazebo_ros_imu_sensor.so" name="imu_plugin">
           <topicName>otto_imu</topicName>
           <bodyName>imu_link</bodyName>
-          <updateRateHZ>200.0</updateRateHZ>
+          <updateRateHZ>2000.0</updateRateHZ>
           <gaussianNoise>0.0</gaussianNoise>
           <xyzOffset>0 0 0</xyzOffset>

Commit message: wtf

File: otto_simulation/urdf/otto-simulation.xacro (robot description, xacro)
@@ -146,5 +146,5 @@
         <origin rpy="${PI/2} 0.0 0.0" xyz="0.0 0.0 0.0"/>
         <geometry>
-            <cylinder radius="0.086" length="0.0001"/>
+            <cylinder radius="0.086" length="0.07"/>
         </geometry>
       </collision>
@@ -292,5 +292,5 @@
         <origin rpy="${PI/2} 0.0 0.0" xyz="0.0 -0.0 0.0"/>
         <geometry>
-            <cylinder radius="0.086" length="0.0001"/>
+            <cylinder radius="0.086" length="0.07"/>
         </geometry>
       </collision>

Commit message: ajarn navigate

File: otto_simulation/urdf/otto-simulation.xacro (robot description, xacro)
@@ -144,7 +144,7 @@
       </visual>
       <collision>
-        <origin rpy="${PI/2} 0.0 0.0" xyz="0.0 0.0 0.0"/>
+        <origin rpy="${PI/2} 0.0 0.0" xyz="0.0 0.02 0.0"/>
         <geometry>
-            <cylinder radius="0.086" length="0.07"/>
+            <cylinder radius="0.086" length="0.03"/>
         </geometry>
       </collision>
@@ -290,7 +290,7 @@
       </visual>
       <collision>
-        <origin rpy="${PI/2} 0.0 0.0" xyz="0.0 -0.0 0.0"/>
+        <origin rpy="${PI/2} 0.0 0.0" xyz="0.0 -0.02 0.0"/>
         <geometry>
-            <cylinder radius="0.086" length="0.07"/>
+            <cylinder radius="0.086" length="0.03"/>
         </geometry>
       </collision>

Commit message: torso task

File: otto_simulation/urdf/otto-simulation.xacro (robot description, xacro)
@@ -172,5 +172,5 @@
       <origin rpy="0.0 0.0 0.0" xyz="0.0 0.055 0.0"/>
       <axis xyz="0.0 1.0 0.0"/>
-      <dynamics damping="0.85" friction="0.05"/>
+      <dynamics damping="0.3" friction="0.05"/>
       <limit effort="10.0" velocity="60"/>
     </joint>
@@ -180,5 +180,5 @@
       <origin rpy="0.0 0.0 0.0" xyz="-0.1414 -0.05 -0.1414"/>
       <axis xyz="0.0 1.0 0.0"/>
-      <dynamics damping="0.85" friction="0.05"/>
+      <dynamics damping="0.3" friction="0.05"/>
       <limit effort="10.0" velocity="60"/>
     </joint>
@@ -318,5 +318,5 @@
       <origin rpy="0.0 0.0 0.0" xyz="0.0 -0.055 0.0"/>
       <axis xyz="0.0 1.0 0.0"/>
-      <dynamics damping="0.85" friction="0.05"/>
+      <dynamics damping="0.3" friction="0.05"/>
       <limit effort="10.0" velocity="60"/>
     </joint>
@@ -326,5 +326,5 @@
       <origin rpy="0.0 0.0 0.0" xyz="-0.1414 0.05 -0.1414"/>
       <axis xyz="0.0 1.0 0.0"/>
-      <dynamics damping="0.85" friction="0.05"/>
+      <dynamics damping="0.3" friction="0.05"/>
       <limit effort="10.0" velocity="60"/>
     </joint>
